File: DR-55-Snare/DR-55-Snare.sch (KiCad schematic (older format))
At the start: 1 part

Commit message: Added drums
Added all drum schematics.
Parts:
- removed R?: R, symbol Device:R
- added C? (x9): C, symbol Device:C
- added D?: D, symbol Device:D
- added Q? (x2): Q_NPN_BCE, symbol Device:Q_NPN_BCE
- added R? (x14): R, symbol Device:R
Connections:
- net labels added: +6V, 6V, GND, NOISEIN, OUT, TRGIN, VOLOUT
- wire segments 0 -> 58
