File: DR-55-Snare/DR-55-Snare.sch (KiCad schematic (older format))
At the start: 26 parts

Commit message: Output finished
Finished the output schematic and routed alll the traces between the submodules
Connections:
- net labels added: NOISYOUT
- net labels removed: VOLOUT
Changed lines of the file:
@@
 $Descr A4 11693 8268
 encoding utf-8
-Sheet 3 7
+Sheet 2 7
 Title ""
 Date ""
@@
 	5000 1000 5000 1100
 Text HLabel 6500 4500 2    50   Input ~ 0
-VOLOUT
+NOISYOUT
 Wire Wire Line
 	6500 4500 6400 4500

Commit message: Values
Added Values to all components
Parts:
- C? (x3): value C -> .0068
- C? (x2): value C -> .0047
- C?: value C -> .0056
- C?: value C -> .001
- C?: value C -> .0022
- C?: value C -> .027
- R? (x2): value R -> 22k
- R?: value R -> 470k
- R? (x2): value R -> 2.2M
- R? (x4): value R -> 10k
- R?: value R -> 180k
- R?: value R -> 330
- R?: value R -> 120k
- R?: value R -> 1M
- R?: value R -> 47k
Changed lines of the file:
@@
 $Descr A4 11693 8268
 encoding utf-8
-Sheet 2 7
+Sheet 7 7
 Title ""
 Date ""
@@
 P 3000 1750
 F 0 "R?" H 3070 1796 50  0000 L CNN
-F 1 "R" H 3070 1705 50  0000 L CNN
+F 1 "22k" H 3070 1705 50  0000 L CNN
 F 2 "" V 2930 1750 50  0001 C CNN
 F 3 "~" H 3000 1750 50  0001 C CNN
@@
 AR Path="/62740CD0/6278054F" Ref="C?"  Part="1"
 F 0 "C?" H 3615 1796 50  0000 L CNN
-F 1 "C" H 3615 1705 50  0000 L CNN
+F 1 ".0068" H 3615 1705 50  0000 L CNN
 F 2 "" H 3538 1600 50  0001 C CNN
 F 3 "~" H 3500 1750 50  0001 C CNN
@@
 P 3500 2250
 F 0 "R?" H 3570 2296 50  0000 L CNN
-F 1 "R" H 3570 2205 50  0000 L CNN
+F 1 "470k" H 3570 2205 50  0000 L CNN
 F 2 "" V 3430 2250 50  0001 C CNN
 F 3 "~" H 3500 2250 50  0001 C CNN
@@
 AR Path="/62740CD0/62781054" Ref="C?"  Part="1"
 F 0 "C?" H 4115 1546 50  0000 L CNN
-F 1 "C" H 4115 1455 50  0000 L CNN
+F 1 ".0068" H 4115 1455 50  0000 L CNN
 F 2 "" H 4038 1350 50  0001 C CNN
 F 3 "~" H 4000 1500 50  0001 C CNN
@@
 AR Path="/62740CD0/627816E5" Ref="C?"  Part="1"
 F 0 "C?" H 4365 2046 50  0000 L CNN
-F 1 "C" H 4365 1955 50  0000 L CNN
+F 1 ".0068" H 4365 1955 50  0000 L CNN
 F 2 "" H 4288 1850 50  0001 C CNN
 F 3 "~" H 4250 2000 50  0001 C CNN
@@
 P 4000 2250
 F 0 "R?" H 4070 2296 50  0000 L CNN
-F 1 "R" H 4070 2205 50  0000 L CNN
+F 1 "22k" H 4070 2205 50  0000 L CNN
 F 2 "" V 3930 2250 50  0001 C CNN
 F 3 "~" H 4000 2250 50  0001 C CNN
@@
 P 4500 1750
 F 0 "R?" H 4570 1796 50  0000 L CNN
-F 1 "R" H 4570 1705 50  0000 L CNN
+F 1 "2.2M" H 4570 1705 50  0000 L CNN
 F 2 "" V 4430 1750 50  0001 C CNN
 F 3 "~" H 4500 1750 50  0001 C CNN
@@
 P 5000 1250
 F 0 "R?" H 5070 1296 50  0000 L CNN
-F 1 "R" H 5070 1205 50  0000 L CNN
+F 1 "10k" H 5070 1205 50  0000 L CNN
 F 2 "" V 4930 1250 50  0001 C CNN
 F 3 "~" H 5000 1250 50  0001 C CNN
@@
 P 5250 1500
 F 0 "R?" H 5320 1546 50  0000 L CNN
-F 1 "R" H 5320 1455 50  0000 L CNN
+F 1 "180k" H 5320 1455 50  0000 L CNN
 F 2 "" V 5180 1500 50  0001 C CNN
 F 3 "~" H 5250 1500 50  0001 C CNN
@@
 AR Path="/62740CD0/627858F7" Ref="C?"  Part="1"
 F 0 "C?" H 5865 1546 50  0000 L CNN
-F 1 "C" H 5865 1455 50  0000 L CNN
+F 1 ".0047" H 5865 1455 50  0000 L CNN
 F 2 "" H 5788 1350 50  0001 C CNN
 F 3 "~" H 5750 1500 50  0001 C CNN
@@
 P 5000 2750
 F 0 "R?" H 5070 2796 50  0000 L CNN
-F 1 "R" H 5070 2705 50  0000 L CNN
+F 1 "330" H 5070 2705 50  0000 L CNN
 F 2 "" V 4930 2750 50  0001 C CNN
 F 3 "~" H 5000 2750 50  0001 C CNN
@@
 P 3500 3250
 F 0 "R?" H 3570 3296 50  0000 L CNN
-F 1 "R" H 3570 3205 50  0000 L CNN
+F 1 "120k" H 3570 3205 50  0000 L CNN
 F 2 "" V 3430 3250 50  0001 C CNN
 F 3 "~" H 3500 3250 50  0001 C CNN
@@
 P 4500 4250
 F 0 "R?" H 4570 4296 50  0000 L CNN
-F 1 "R" H 4570 4205 50  0000 L CNN
+F 1 "10k" H 4570 4205 50  0000 L CNN
 F 2 "" V 4430 4250 50  0001 C CNN
 F 3 "~" H 4500 4250 50  0001 C CNN
@@
 P 4500 4750
 F 0 "R?" H 4570 4796 50  0000 L CNN
-F 1 "R" H 4570 4705 50  0000 L CNN
+F 1 "1M" H 4570 4705 50  0000 L CNN
 F 2 "" V 4430 4750 50  0001 C CNN
 F 3 "~" H 4500 4750 50  0001 C CNN
@@
 P 4250 4500
 F 0 "R?" H 4320 4546 50  0000 L CNN
-F 1 "R" H 4320 4455 50  0000 L CNN
+F 1 "2.2M" H 4320 4455 50  0000 L CNN
 F 2 "" V 4180 4500 50  0001 C CNN
 F 3 "~" H 4250 4500 50  0001 C CNN
@@
 P 5000 3750
 F 0 "R?" H 5070 3796 50  0000 L CNN
-F 1 "R" H 5070 3705 50  0000 L CNN
+F 1 "10k" H 5070 3705 50  0000 L CNN
 F 2 "" V 4930 3750 50  0001 C CNN
 F 3 "~" H 5000 3750 50  0001 C CNN
@@
 P 5750 4000
 F 0 "R?" H 5820 4046 50  0000 L CNN
-F 1 "R" H 5820 3955 50  0000 L CNN
+F 1 "10k" H 5820 3955 50  0000 L CNN
 F 2 "" V 5680 4000 50  0001 C CNN
 F 3 "~" H 5750 4000 50  0001 C CNN
@@
 P 5750 4500
 F 0 "R?" H 5820 4546 50  0000 L CNN
-F 1 "R" H 5820 4455 50  0000 L CNN
+F 1 "47k" H 5820 4455 50  0000 L CNN
 F 2 "" V 5680 4500 50  0001 C CNN
 F 3 "~" H 5750 4500 50  0001 C CNN
@@
 AR Path="/62740CD0/627A13BD" Ref="C?"  Part="1"
 F 0 "C?" H 5615 3796 50  0000 L CNN
-F 1 "C" H 5615 3705 50  0000 L CNN
+F 1 ".0056" H 5615 3705 50  0000 L CNN
 F 2 "" H 5538 3600 50  0001 C CNN
 F 3 "~" H 5500 3750 50  0001 C CNN
@@
 AR Path="/62740CD0/627A1D3D" Ref="C?"  Part="1"
 F 0 "C?" H 6365 4046 50  0000 L CNN
-F 1 "C" H 6365 3955 50  0000 L CNN
+F 1 ".0047" H 6365 3955 50  0000 L CNN
 F 2 "" H 6288 3850 50  0001 C CNN
 F 3 "~" H 6250 4000 50  0001 C CNN
@@
 AR Path="/62740CD0/627A20BC" Ref="C?"  Part="1"
 F 0 "C?" H 6365 4546 50  0000 L CNN
-F 1 "C" H 6365 4455 50  0000 L CNN
+F 1 ".001" H 6365 4455 50  0000 L CNN
 F 2 "" H 6288 4350 50  0001 C CNN
 F 3 "~" H 6250 4500 50  0001 C CNN
@@
 AR Path="/62740CD0/627A29DF" Ref="C?"  Part="1"
 F 0 "C?" H 4365 4046 50  0000 L CNN
-F 1 "C" H 4365 3955 50  0000 L CNN
+F 1 ".0022" H 4365 3955 50  0000 L CNN
 F 2 "" H 4288 3850 50  0001 C CNN
 F 3 "~" H 4250 4000 50  0001 C CNN
@@
 AR Path="/62740CD0/627A309A" Ref="C?"  Part="1"
 F 0 "C?" H 3615 4796 50  0000 L CNN
-F 1 "C" H 3615 4705 50  0000 L CNN
+F 1 ".027" H 3615 4705 50  0000 L CNN
 F 2 "" H 3538 4600 50  0001 C CNN
 F 3 "~" H 3500 4750 50  0001 C CNN

Commit message: Resistor enumeration
All resistors, diodes and transistors get numbers
Parts:
- gave numbers to parts that had none: 15
Changed lines of the file:
@@
 $Descr A4 11693 8268
 encoding utf-8
-Sheet 7 7
+Sheet 6 7
 Title ""
 Date ""
@@
 TRGIN
 $Comp
-L Device:R R?
+L Device:R R29
 U 1 1 6277F393
 P 3000 1750
-F 0 "R?" H 3070 1796 50  0000 L CNN
+F 0 "R29" H 3070 1796 50  0000 L CNN
 F 1 "22k" H 3070 1705 50  0000 L CNN
 F 2 "" V 2930 1750 50  0001 C CNN
@@
 $EndComp
 $Comp
-L Device:R R?
+L Device:R R30
 U 1 1 62780875
 P 3500 2250
-F 0 "R?" H 3570 2296 50  0000 L CNN
+F 0 "R30" H 3570 2296 50  0000 L CNN
 F 1 "470k" H 3570 2205 50  0000 L CNN
 F 2 "" V 3430 2250 50  0001 C CNN
@@
 $EndComp
 $Comp
-L Device:R R?
+L Device:R R28
 U 1 1 62781A4A
 P 4000 2250
-F 0 "R?" H 4070 2296 50  0000 L CNN
+F 0 "R28" H 4070 2296 50  0000 L CNN
 F 1 "22k" H 4070 2205 50  0000 L CNN
 F 2 "" V 3930 2250 50  0001 C CNN
@@
 	4400 2000 4500 2000
 $Comp
-L Device:R R?
+L Device:R R28
 U 1 1 627831BE
 P 4500 1750
-F 0 "R?" H 4570 1796 50  0000 L CNN
+F 0 "R28" H 4570 1796 50  0000 L CNN
 F 1 "2.2M" H 4570 1705 50  0000 L CNN
 F 2 "" V 4430 1750 50  0001 C CNN
@@
 P 4900 2000
 AR Path="/6276643A/62783C78" Ref="Q?"  Part="1"
-AR Path="/62740CD0/62783C78" Ref="Q?"  Part="1"
-F 0 "Q?" H 5091 2046 50  0000 L CNN
+AR Path="/62740CD0/62783C78" Ref="Q10"  Part="1"
+F 0 "Q10" H 5091 2046 50  0000 L CNN
 F 1 "Q_NPN_BCE" H 5091 1955 50  0000 L CNN
 F 2 "" H 5100 2100 50  0001 C CNN
@@
 Connection ~ 4500 1500
 $Comp
-L Device:R R?
+L Device:R R25
 U 1 1 62784858
 P 5000 1250
-F 0 "R?" H 5070 1296 50  0000 L CNN
+F 0 "R25" H 5070 1296 50  0000 L CNN
 F 1 "10k" H 5070 1205 50  0000 L CNN
 F 2 "" V 4930 1250 50  0001 C CNN
@@
 Connection ~ 5000 1500
 $Comp
-L Device:R R?
+L Device:R R26
 U 1 1 627852F6
 P 5250 1500
-F 0 "R?" H 5320 1546 50  0000 L CNN
+F 0 "R26" H 5320 1546 50  0000 L CNN
 F 1 "180k" H 5320 1455 50  0000 L CNN
 F 2 "" V 5180 1500 50  0001 C CNN
@@
 	5600 1500 5400 1500
 $Comp
-L Device:R R?
+L Device:R R27
 U 1 1 62786408
 P 5000 2750
-F 0 "R?" H 5070 2796 50  0000 L CNN
+F 0 "R27" H 5070 2796 50  0000 L CNN
 F 1 "330" H 5070 2705 50  0000 L CNN
 F 2 "" V 4930 2750 50  0001 C CNN
@@
 	3500 2600 3500 2500
 $Comp
-L Device:R R?
+L Device:R R32
 U 1 1 6278AF7C
 P 3500 3250
-F 0 "R?" H 3570 3296 50  0000 L CNN
+F 0 "R32" H 3570 3296 50  0000 L CNN
 F 1 "120k" H 3570 3205 50  0000 L CNN
 F 2 "" V 3430 3250 50  0001 C CNN
@@
 	3500 3100 3500 2900
 $Comp
-L Device:R R?
+L Device:R R35
 U 1 1 6279E0D3
 P 4500 4250
-F 0 "R?" H 4570 4296 50  0000 L CNN
+F 0 "R35" H 4570 4296 50  0000 L CNN
 F 1 "10k" H 4570 4205 50  0000 L CNN
 F 2 "" V 4430 4250 50  0001 C CNN
@@
 $EndComp
 $Comp
-L Device:R R?
+L Device:R R34
 U 1 1 6279E744
 P 4500 4750
-F 0 "R?" H 4570 4796 50  0000 L CNN
+F 0 "R34" H 4570 4796 50  0000 L CNN
 F 1 "1M" H 4570 4705 50  0000 L CNN
 F 2 "" V 4430 4750 50  0001 C CNN
@@
 $EndComp
 $Comp
-L Device:R R?
+L Device:R R33
 U 1 1 6279EBC2
 P 4250 4500
-F 0 "R?" H 4320 4546 50  0000 L CNN
+F 0 "R33" H 4320 4546 50  0000 L CNN
 F 1 "2.2M" H 4320 4455 50  0000 L CNN
 F 2 "" V 4180 4500 50  0001 C CNN
@@
 $EndComp
 $Comp
-L Device:R R?
+L Device:R R36
 U 1 1 6279FD82
 P 5000 3750
-F 0 "R?" H 5070 3796 50  0000 L CNN
+F 0 "R36" H 5070 3796 50  0000 L CNN
 F 1 "10k" H 5070 3705 50  0000 L CNN
 F 2 "" V 4930 3750 50  0001 C CNN
@@
 $EndComp
 $Comp
-L Device:R R?
+L Device:R R37
 U 1 1 627A046A
 P 5750 4000
-F 0 "R?" H 5820 4046 50  0000 L CNN
+F 0 "R37" H 5820 4046 50  0000 L CNN
 F 1 "10k" H 5820 3955 50  0000 L CNN
 F 2 "" V 5680 4000 50  0001 C CNN
@@
 $EndComp
 $Comp
-L Device:R R?
+L Device:R R38
 U 1 1 627A08AF
 P 5750 4500
-F 0 "R?" H 5820 4546 50  0000 L CNN
+F 0 "R38" H 5820 4546 50  0000 L CNN
 F 1 "47k" H 5820 4455 50  0000 L CNN
 F 2 "" V 5680 4500 50  0001 C CNN
@@
 P 4900 4500
 AR Path="/6276643A/627A3A39" Ref="Q?"  Part="1"
-AR Path="/62740CD0/627A3A39" Ref="Q?"  Part="1"
-F 0 "Q?" H 5091 4546 50  0000 L CNN
+AR Path="/62740CD0/627A3A39" Ref="Q11"  Part="1"
+F 0 "Q11" H 5091 4546 50  0000 L CNN
 F 1 "Q_NPN_BCE" H 5091 4455 50  0000 L CNN
 F 2 "" H 5100 4600 50  0001 C CNN

Commit message: Footprints added
Added most of the footprints for a 0805 SMD PCB. some placeholder footprints added and some missing
Parts:
- C15, C19, C20, C21, C22, C23, C?16, C?17, C?18: renamed from C?; footprint (none) -> Capacitor_SMD:C_0805_2012Metric_Pad1.18x1.45mm_HandSolder
- D3: renamed from D?; footprint (none) -> Diode_SMD:D_SOD-123
- Q10, Q11: footprint (none) -> Package_TO_SOT_SMD:SOT-23
- R25, R26, R27, R28, R29, R30, R32, R33, R34, R35, R36, R37, R38: footprint (none) -> Resistor_SMD:R_0805_2012Metric_Pad1.20x1.40mm_HandSolder
- R281: renamed from R28; footprint (none) -> Resistor_SMD:R_0805_2012Metric_Pad1.20x1.40mm_HandSolder

Commit message: changed some stuff
Parts:
- C15, C19, C20, C21, C22, C23, C?16, C?17, C?18: footprint Capacitor_SMD:C_0805_2012Metric_Pad1.18x1.45mm_HandSolder -> Capacitor_SMD:C_0805_2012Metric
- D3: footprint Diode_SMD:D_SOD-123 -> Diode_SMD:D_SOD-123F
- Q10, Q11: footprint Package_TO_SOT_SMD:SOT-23 -> Package_TO_SOT_SMD:SOT-89-3
- R25, R26, R27, R28, R281, R29, R30, R32, R33, R34, R35, R36, R37, R38: footprint Resistor_SMD:R_0805_2012Metric_Pad1.20x1.40mm_HandSolder -> Resistor_SMD:R_0805_2012Metric
Changed lines of the file:
@@
 $Descr A4 11693 8268
 encoding utf-8
-Sheet 6 7
+Sheet 6 8
 Title ""
 Date ""
@@
 F 0 "R29" H 3070 1796 50  0000 L CNN
 F 1 "22k" H 3070 1705 50  0000 L CNN
-F 2 "Resistor_SMD:R_0805_2012Metric_Pad1.20x1.40mm_HandSolder" V 2930 1750 50  0001 C CNN
+F 2 "Resistor_SMD:R_0805_2012Metric" V 2930 1750 50  0001 C CNN
 F 3 "~" H 3000 1750 50  0001 C CNN
 	1    3000 1750
@@
 F 0 "C?16" H 3615 1796 50  0000 L CNN
 F 1 ".0068" H 3615 1705 50  0000 L CNN
-F 2 "Capacitor_SMD:C_0805_2012Metric_Pad1.18x1.45mm_HandSolder" H 3538 1600 50  0001 C CNN
+F 2 "Capacitor_SMD:C_0805_2012Metric" H 3538 1600 50  0001 C CNN
 F 3 "~" H 3500 1750 50  0001 C CNN
 	1    3500 1750
@@
 F 0 "R30" H 3570 2296 50  0000 L CNN
 F 1 "470k" H 3570 2205 50  0000 L CNN
-F 2 "Resistor_SMD:R_0805_2012Metric_Pad1.20x1.40mm_HandSolder" V 3430 2250 50  0001 C CNN
+F 2 "Resistor_SMD:R_0805_2012Metric" V 3430 2250 50  0001 C CNN
 F 3 "~" H 3500 2250 50  0001 C CNN
 	1    3500 2250
@@
 F 0 "C?17" H 4115 1546 50  0000 L CNN
 F 1 ".0068" H 4115 1455 50  0000 L CNN
-F 2 "Capacitor_SMD:C_0805_2012Metric_Pad1.18x1.45mm_HandSolder" H 4038 1350 50  0001 C CNN
+F 2 "Capacitor_SMD:C_0805_2012Metric" H 4038 1350 50  0001 C CNN
 F 3 "~" H 4000 1500 50  0001 C CNN
 	1    4000 1500
@@
 F 0 "C15" H 4365 2046 50  0000 L CNN
 F 1 ".0068" H 4365 1955 50  0000 L CNN
-F 2 "Capacitor_SMD:C_0805_2012Metric_Pad1.18x1.45mm_HandSolder" H 4288 1850 50  0001 C CNN
+F 2 "Capacitor_SMD:C_0805_2012Metric" H 4288 1850 50  0001 C CNN
 F 3 "~" H 4250 2000 50  0001 C CNN
 	1    4250 2000
@@
 F 0 "R281" H 4070 2296 50  0000 L CNN
 F 1 "22k" H 4070 2205 50  0000 L CNN
-F 2 "Resistor_SMD:R_0805_2012Metric_Pad1.20x1.40mm_HandSolder" V 3930 2250 50  0001 C CNN
+F 2 "Resistor_SMD:R_0805_2012Metric" V 3930 2250 50  0001 C CNN
 F 3 "~" H 4000 2250 50  0001 C CNN
 	1    4000 2250
@@
 F 0 "R28" H 4570 1796 50  0000 L CNN
 F 1 "2.2M" H 4570 1705 50  0000 L CNN
-F 2 "Resistor_SMD:R_0805_2012Metric_Pad1.20x1.40mm_HandSolder" V 4430 1750 50  0001 C CNN
+F 2 "Resistor_SMD:R_0805_2012Metric" V 4430 1750 50  0001 C CNN
 F 3 "~" H 4500 1750 50  0001 C CNN
 	1    4500 1750
@@
 F 0 "Q10" H 5091 2046 50  0000 L CNN
 F 1 "Q_NPN_BCE" H 5091 1955 50  0000 L CNN
-F 2 "Package_TO_SOT_SMD:SOT-23" H 5100 2100 50  0001 C CNN
+F 2 "Package_TO_SOT_SMD:SOT-89-3" H 5100 2100 50  0001 C CNN
 F 3 "~" H 4900 2000 50  0001 C CNN
 	1    4900 2000
@@
 F 0 "R25" H 5070 1296 50  0000 L CNN
 F 1 "10k" H 5070 1205 50  0000 L CNN
-F 2 "Resistor_SMD:R_0805_2012Metric_Pad1.20x1.40mm_HandSolder" V 4930 1250 50  0001 C CNN
+F 2 "Resistor_SMD:R_0805_2012Metric" V 4930 1250 50  0001 C CNN
 F 3 "~" H 5000 1250 50  0001 C CNN
 	1    5000 1250
@@
 F 0 "R26" H 5320 1546 50  0000 L CNN
 F 1 "180k" H 5320 1455 50  0000 L CNN
-F 2 "Resistor_SMD:R_0805_2012Metric_Pad1.20x1.40mm_HandSolder" V 5180 1500 50  0001 C CNN
+F 2 "Resistor_SMD:R_0805_2012Metric" V 5180 1500 50  0001 C CNN
 F 3 "~" H 5250 1500 50  0001 C CNN
 	1    5250 1500
@@
 F 0 "C?18" H 5865 1546 50  0000 L CNN
 F 1 ".0047" H 5865 1455 50  0000 L CNN
-F 2 "Capacitor_SMD:C_0805_2012Metric_Pad1.18x1.45mm_HandSolder" H 5788 1350 50  0001 C CNN
+F 2 "Capacitor_SMD:C_0805_2012Metric" H 5788 1350 50  0001 C CNN
 F 3 "~" H 5750 1500 50  0001 C CNN
 	1    5750 1500
@@
 F 0 "R27" H 5070 2796 50  0000 L CNN
 F 1 "330" H 5070 2705 50  0000 L CNN
-F 2 "Resistor_SMD:R_0805_2012Metric_Pad1.20x1.40mm_HandSolder" V 4930 2750 50  0001 C CNN
+F 2 "Resistor_SMD:R_0805_2012Metric" V 4930 2750 50  0001 C CNN
 F 3 "~" H 5000 2750 50  0001 C CNN
 	1    5000 2750
@@
 F 0 "D3" V 3546 2670 50  0000 R CNN
 F 1 "D" V 3455 2670 50  0000 R CNN
-F 2 "Diode_SMD:D_SOD-123" H 3500 2750 50  0001 C CNN
+F 2 "Diode_SMD:D_SOD-123F" H 3500 2750 50  0001 C CNN
 F 3 "~" H 3500 2750 50  0001 C CNN
 	1    3500 2750
@@
 F 0 "R32" H 3570 3296 50  0000 L CNN
 F 1 "120k" H 3570 3205 50  0000 L CNN
-F 2 "Resistor_SMD:R_0805_2012Metric_Pad1.20x1.40mm_HandSolder" V 3430 3250 50  0001 C CNN
+F 2 "Resistor_SMD:R_0805_2012Metric" V 3430 3250 50  0001 C CNN
 F 3 "~" H 3500 3250 50  0001 C CNN
 	1    3500 3250
@@
 F 0 "R35" H 4570 4296 50  0000 L CNN
 F 1 "10k" H 4570 4205 50  0000 L CNN
-F 2 "Resistor_SMD:R_0805_2012Metric_Pad1.20x1.40mm_HandSolder" V 4430 4250 50  0001 C CNN
+F 2 "Resistor_SMD:R_0805_2012Metric" V 4430 4250 50  0001 C CNN
 F 3 "~" H 4500 4250 50  0001 C CNN
 	1    4500 4250
@@
 F 0 "R34" H 4570 4796 50  0000 L CNN
 F 1 "1M" H 4570 4705 50  0000 L CNN
-F 2 "Resistor_SMD:R_0805_2012Metric_Pad1.20x1.40mm_HandSolder" V 4430 4750 50  0001 C CNN
+F 2 "Resistor_SMD:R_0805_2012Metric" V 4430 4750 50  0001 C CNN
 F 3 "~" H 4500 4750 50  0001 C CNN
 	1    4500 4750
@@
 F 0 "R33" H 4320 4546 50  0000 L CNN
 F 1 "2.2M" H 4320 4455 50  0000 L CNN
-F 2 "Resistor_SMD:R_0805_2012Metric_Pad1.20x1.40mm_HandSolder" V 4180 4500 50  0001 C CNN
+F 2 "Resistor_SMD:R_0805_2012Metric" V 4180 4500 50  0001 C CNN
 F 3 "~" H 4250 4500 50  0001 C CNN
 	1    4250 4500
@@
 F 0 "R36" H 5070 3796 50  0000 L CNN
 F 1 "10k" H 5070 3705 50  0000 L CNN
-F 2 "Resistor_SMD:R_0805_2012Metric_Pad1.20x1.40mm_HandSolder" V 4930 3750 50  0001 C CNN
+F 2 "Resistor_SMD:R_0805_2012Metric" V 4930 3750 50  0001 C CNN
 F 3 "~" H 5000 3750 50  0001 C CNN
 	1    5000 3750
@@
 F 0 "R37" H 5820 4046 50  0000 L CNN
 F 1 "10k" H 5820 3955 50  0000 L CNN
-F 2 "Resistor_SMD:R_0805_2012Metric_Pad1.20x1.40mm_HandSolder" V 5680 4000 50  0001 C CNN
+F 2 "Resistor_SMD:R_0805_2012Metric" V 5680 4000 50  0001 C CNN
 F 3 "~" H 5750 4000 50  0001 C CNN
 	1    5750 4000
@@
 F 0 "R38" H 5820 4546 50  0000 L CNN
 F 1 "47k" H 5820 4455 50  0000 L CNN
-F 2 "Resistor_SMD:R_0805_2012Metric_Pad1.20x1.40mm_HandSolder" V 5680 4500 50  0001 C CNN
+F 2 "Resistor_SMD:R_0805_2012Metric" V 5680 4500 50  0001 C CNN
 F 3 "~" H 5750 4500 50  0001 C CNN
 	1    5750 4500
@@
 F 0 "C20" H 5615 3796 50  0000 L CNN
 F 1 ".0056" H 5615 3705 50  0000 L CNN
-F 2 "Capacitor_SMD:C_0805_2012Metric_Pad1.18x1.45mm_HandSolder" H 5538 3600 50  0001 C CNN
+F 2 "Capacitor_SMD:C_0805_2012Metric" H 5538 3600 50  0001 C CNN
 F 3 "~" H 5500 3750 50  0001 C CNN
 	1    5500 3750
@@
 F 0 "C21" H 6365 4046 50  0000 L CNN
 F 1 ".0047" H 6365 3955 50  0000 L CNN
-F 2 "Capacitor_SMD:C_0805_2012Metric_Pad1.18x1.45mm_HandSolder" H 6288 3850 50  0001 C CNN
+F 2 "Capacitor_SMD:C_0805_2012Metric" H 6288 3850 50  0001 C CNN
 F 3 "~" H 6250 4000 50  0001 C CNN
 	1    6250 4000
@@
 F 0 "C22" H 6365 4546 50  0000 L CNN
 F 1 ".001" H 6365 4455 50  0000 L CNN
-F 2 "Capacitor_SMD:C_0805_2012Metric_Pad1.18x1.45mm_HandSolder" H 6288 4350 50  0001 C CNN
+F 2 "Capacitor_SMD:C_0805_2012Metric" H 6288 4350 50  0001 C CNN
 F 3 "~" H 6250 4500 50  0001 C CNN
 	1    6250 4500
@@
 F 0 "C23" H 4365 4046 50  0000 L CNN
 F 1 ".0022" H 4365 3955 50  0000 L CNN
-F 2 "Capacitor_SMD:C_0805_2012Metric_Pad1.18x1.45mm_HandSolder" H 4288 3850 50  0001 C CNN
+F 2 "Capacitor_SMD:C_0805_2012Metric" H 4288 3850 50  0001 C CNN
 F 3 "~" H 4250 4000 50  0001 C CNN
 	1    4250 4000
@@
 F 0 "C19" H 3615 4796 50  0000 L CNN
 F 1 ".027" H 3615 4705 50  0000 L CNN
-F 2 "Capacitor_SMD:C_0805_2012Metric_Pad1.18x1.45mm_HandSolder" H 3538 4600 50  0001 C CNN
+F 2 "Capacitor_SMD:C_0805_2012Metric" H 3538 4600 50  0001 C CNN
 F 3 "~" H 3500 4750 50  0001 C CNN
 	1    3500 4750
@@
 F 0 "Q11" H 5091 4546 50  0000 L CNN
 F 1 "Q_NPN_BCE" H 5091 4455 50  0000 L CNN
-F 2 "Package_TO_SOT_SMD:SOT-23" H 5100 4600 50  0001 C CNN
+F 2 "Package_TO_SOT_SMD:SOT-89-3" H 5100 4600 50  0001 C CNN
 F 3 "~" H 4900 4500 50  0001 C CNN
 	1    4900 4500
