File: DR-55/DR-55.kicad_pcb (KiCad board)
At the start: 2 copper layers, 100 x 100 mm, 123 parts, among them J1 KICK, J2 SNARE, J3 RIM, J4 HIHAT, J5 ACCENT, J6 OUT, J7 Accent OUT, Q1 Q_NPN_BCE, Q10 Q_NPN_BCE, Q11 Q_NPN_BCE, Q12 Q_NPN_BCE, Q2 Q_NPN_BCE, Q3 Q_NJFET_SGD, Q4 Q_NPN_BCE, Q6 Q_NPN_BCE, Q7 Q_NPN_BCE, Q8 Q_NPN_BCE, Q9 Q_NPN_BCE

Commit message: changed some stuff
Parts:
- removed J7: Accent OUT, Connector_PinHeader_2.54mm:PinHeader_1x03_P2.54mm_Vertical
- added C101: 100n, Capacitor_SMD:C_0805_2012Metric, F.Cu at (28.0, -8.50)
- added C102: 100n, Capacitor_SMD:C_0805_2012Metric, F.Cu at (28.0, -1.00)
- added D101: D, Diode_SMD:D_SOD-123F, F.Cu at (32.0, -8.50)
- added D102: D, Diode_SMD:D_SOD-123F, F.Cu at (32.0, -1.00)
- added J100: Conn_02x05_Odd_Even, Connector_PinSocket_2.54mm:PinSocket_2x05_P2.54mm_Vertical, B.Cu at (26.5, -3.50)
- added R110: 100k, Resistor_SMD:R_0805_2012Metric, F.Cu at (21.5, -3.00)
- added R120: 100k, Resistor_SMD:R_0805_2012Metric, F.Cu at (21.5, -6.50)
- C1, C10, C15, C19, C2, C20, C21, C22, C23, C25, C27, C28, C29, C3, C30, C31, C32, C33, C34, C35, C36, C37, C38, C4, C5, C?16, C?17, C?18, C?26: footprint Capacitor_SMD:C_0805_2012Metric_Pad1.18x1.45mm_HandSolder -> Capacitor_SMD:C_0805_2012Metric
- C11, C12, C14, C24, C6, C7, C8, C9: footprint Connector_PinHeader_2.54mm:PinHeader_1x02_P2.54mm_Vertical -> Capacitor_THT:CP_Radial_D5.0mm_P2.50mm
- D2, D3, D4: footprint Diode_SMD:D_SOD-123 -> Diode_SMD:D_SOD-123F
- J1, J2, J3, J4, J5, J6: footprint Connector_PinHeader_2.54mm:PinHeader_1x03_P2.54mm_Vertical -> eurocad-master:PJ301M-12
- Q1, Q10, Q11, Q12, Q2, Q4, Q6, Q7, Q8, Q9: footprint Package_TO_SOT_SMD:SOT-23 -> Package_TO_SOT_SMD:SOT-89-3
- Q3: footprint Connector_PinHeader_2.54mm:PinHeader_1x03_P2.54mm_Vertical -> Package_TO_SOT_THT:TO-92L_HandSolder
- R1, R10, R101, R102, R11, R12, R13, R14, R15, R16, R17, R18, R19, R2, R20, R21, R22, R24, R25, R26, R27, R28, R281, R29, R30, R32, R33, R34, R35, R36, R37, R38, R39, R4, R40, R41, R42, R43, R44, R45, R46, R47, R48, R49, R5, R50, R51, R52, R53, R54, R55, R56, R57, R59, R6, R60, R7, R8, R9: footprint Resistor_SMD:R_0805_2012Metric_Pad1.20x1.40mm_HandSolder -> Resistor_SMD:R_0805_2012Metric
- VR1, VR2, VR4: footprint Connector_PinHeader_2.54mm:PinHeader_1x03_P2.54mm_Vertical -> Potentiometer_THT:Potentiometer_Alpha_RD901F-40-00D_Single_Vertical
- VR7: footprint Connector_PinHeader_2.54mm:PinHeader_1x03_P2.54mm_Vertical -> Potentiometer_THT:Potentiometer_Bourns_3339P_Vertical_HandSoldering
- moved C25 299.3 mm to (-30.2, -25.6)
- moved VR7 296.8 mm to (-32.3, -9.96), turned to 0 degrees
- moved Q6 294.0 mm to (-29.3, -33.5), turned to 0 degrees
- moved C34 287.2 mm to (-34.7, -6.38), turned to 0 degrees
- moved R43 285.5 mm to (-15.1, -32.1), turned to 0 degrees
- moved R51 285.0 mm to (-30.3, -6.41), turned to 0 degrees
- moved C14 284.9 mm to (-25.6, -13.8), turned to 0 degrees
- moved R41 283.7 mm to (-16.9, -26.1)
- moved C31 282.6 mm to (-19.6, -35.0)
- moved D4 281.2 mm to (-29.6, -28.8), turned to 0 degrees
- moved C30 281.1 mm to (-24.7, -28.9)
- moved R42 280.8 mm to (-15.9, -29.1), turned to 0 degrees
- moved Q9 280.0 mm to (-18.0, -14.1)
- moved R44 279.8 mm to (-21.3, -26.0), turned to 0 degrees
- moved C29 278.5 mm to (-24.0, -32.0)
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Routing:
- net GND: track 246.6 -> 91.3 mm
- net +6V: track 57.5 -> 3.69 mm, vias 2 -> 0
- net /Snare/TRGIN: track 25.6 -> 0.00 mm, vias 1 -> 0
- net /OUTPUT/ACCENT-IN: track 20.4 -> 0.00 mm, vias 2 -> 0
- net Net-(D2-Pad1): track 18.7 -> 0.00 mm
- net Net-(C29-Pad2): track 18.3 -> 0.00 mm
- net /OUTPUT/OUT: track 16.3 -> 0.00 mm
- net Net-(C12-Pad1): track 16.1 -> 0.00 mm
- net Net-(C102-Pad1): track 0.00 -> 12.5 mm
- net /OUTPUT/TRGIN: track 12.5 -> 0.00 mm
- net Net-(D102-Pad2): track 0.00 -> 10.5 mm
- net Net-(C31-Pad2): track 8.97 -> 0.00 mm
- net /Rim Shot/TRGIN: track 8.91 -> 0.00 mm
- net Net-(C1-Pad1): track 20.6 -> 11.9 mm
- net /Kick/TRGIN: track 8.21 -> 0.00 mm
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Other:
- board size 100 x 100 mm -> 40 x 105 mm
- board text removed: "Kick"
- board text removed: "Snare"
