File: DR-55-Hats/DR-55-Hats.sch (KiCad schematic (older format))
At the start: 16 parts

Commit message: Output finished
Finished the output schematic and routed alll the traces between the submodules
Connections:
- net labels added: NOISYOUT
- net labels removed: VOLOUT
Changed lines of the file:
@@
 OUT
 Text HLabel 8000 4000 2    50   Input ~ 0
-VOLOUT
+NOISYOUT
 Text HLabel 5000 2650 0    50   Input ~ 0
 6V

Commit message: Values
Added Values to all components
Parts:
- C?: value C -> .047
- C?: value C -> .018
- C? (x2): value C -> .001
- C?: value C -> .0068
- C?: value C -> .0022
- L?: value L -> 45mH
- R? (x2): value R -> 1M
- R?: value R -> 82k
- R?: value R -> 2.2M
- R? (x2): value R -> 10k
- R?: value R -> 47k
Changed lines of the file:
@@
 $Descr A4 11693 8268
 encoding utf-8
-Sheet 3 7
+Sheet 2 7
 Title ""
 Date ""
@@
 AR Path="/627D8A3A/627E8B98" Ref="C?"  Part="1"
 F 0 "C?" H 4365 3046 50  0000 L CNN
-F 1 "C" H 4365 2955 50  0000 L CNN
+F 1 ".047" H 4365 2955 50  0000 L CNN
 F 2 "" H 4288 2850 50  0001 C CNN
 F 3 "~" H 4250 3000 50  0001 C CNN
@@
 AR Path="/627D8A3A/627E8F93" Ref="R?"  Part="1"
 F 0 "R?" H 4570 3296 50  0000 L CNN
-F 1 "R" H 4570 3205 50  0000 L CNN
+F 1 "1M" H 4570 3205 50  0000 L CNN
 F 2 "" V 4430 3250 50  0001 C CNN
 F 3 "~" H 4500 3250 50  0001 C CNN
@@
 AR Path="/627D8A3A/627E91C5" Ref="R?"  Part="1"
 F 0 "R?" H 5070 3796 50  0000 L CNN
-F 1 "R" H 5070 3705 50  0000 L CNN
+F 1 "82k" H 5070 3705 50  0000 L CNN
 F 2 "" V 4930 3750 50  0001 C CNN
 F 3 "~" H 5000 3750 50  0001 C CNN
@@
 AR Path="/627D8A3A/627E9A1B" Ref="R?"  Part="1"
 F 0 "R?" H 5320 4046 50  0000 L CNN
-F 1 "R" H 5320 3955 50  0000 L CNN
+F 1 "2.2M" H 5320 3955 50  0000 L CNN
 F 2 "" V 5180 4000 50  0001 C CNN
 F 3 "~" H 5250 4000 50  0001 C CNN
@@
 AR Path="/627D8A3A/627EA05F" Ref="C?"  Part="1"
 F 0 "C?" H 5115 4296 50  0000 L CNN
-F 1 "C" H 5115 4205 50  0000 L CNN
+F 1 ".018" H 5115 4205 50  0000 L CNN
 F 2 "" H 5038 4100 50  0001 C CNN
 F 3 "~" H 5000 4250 50  0001 C CNN
@@
 AR Path="/627D8A3A/627EA305" Ref="R?"  Part="1"
 F 0 "R?" H 5570 4296 50  0000 L CNN
-F 1 "R" H 5570 4205 50  0000 L CNN
+F 1 "1M" H 5570 4205 50  0000 L CNN
 F 2 "" V 5430 4250 50  0001 C CNN
 F 3 "~" H 5500 4250 50  0001 C CNN
@@
 AR Path="/627D8A3A/627EAA10" Ref="R?"  Part="1"
 F 0 "R?" H 5570 3296 50  0000 L CNN
-F 1 "R" H 5570 3205 50  0000 L CNN
+F 1 "10k" H 5570 3205 50  0000 L CNN
 F 2 "" V 5430 3250 50  0001 C CNN
 F 3 "~" H 5500 3250 50  0001 C CNN
@@
 AR Path="/627D8A3A/627EADD0" Ref="C?"  Part="1"
 F 0 "C?" H 5615 2796 50  0000 L CNN
-F 1 "C" H 5615 2705 50  0000 L CNN
+F 1 ".001" H 5615 2705 50  0000 L CNN
 F 2 "" H 5538 2600 50  0001 C CNN
 F 3 "~" H 5500 2750 50  0001 C CNN
@@
 P 6000 3250
 F 0 "L?" H 6053 3296 50  0000 L CNN
-F 1 "L" H 6053 3205 50  0000 L CNN
+F 1 "45mH" H 6053 3205 50  0000 L CNN
 F 2 "" H 6000 3250 50  0001 C CNN
 F 3 "~" H 6000 3250 50  0001 C CNN
@@
 AR Path="/627D8A3A/627ECA20" Ref="C?"  Part="1"
 F 0 "C?" H 6615 3296 50  0000 L CNN
-F 1 "C" H 6615 3205 50  0000 L CNN
+F 1 ".0068" H 6615 3205 50  0000 L CNN
 F 2 "" H 6538 3100 50  0001 C CNN
 F 3 "~" H 6500 3250 50  0001 C CNN
@@
 P 6750 3500
 F 0 "R?" H 6820 3546 50  0000 L CNN
-F 1 "R" H 6820 3455 50  0000 L CNN
+F 1 "10k" H 6820 3455 50  0000 L CNN
 F 2 "" V 6680 3500 50  0001 C CNN
 F 3 "~" H 6750 3500 50  0001 C CNN
@@
 P 6750 4000
 F 0 "R?" H 6820 4046 50  0000 L CNN
-F 1 "R" H 6820 3955 50  0000 L CNN
+F 1 "47k" H 6820 3955 50  0000 L CNN
 F 2 "" V 6680 4000 50  0001 C CNN
 F 3 "~" H 6750 4000 50  0001 C CNN
@@
 AR Path="/627D8A3A/627F04D0" Ref="C?"  Part="1"
 F 0 "C?" H 7365 3546 50  0000 L CNN
-F 1 "C" H 7365 3455 50  0000 L CNN
+F 1 ".0022" H 7365 3455 50  0000 L CNN
 F 2 "" H 7288 3350 50  0001 C CNN
 F 3 "~" H 7250 3500 50  0001 C CNN
@@
 AR Path="/627D8A3A/627F04D6" Ref="C?"  Part="1"
 F 0 "C?" H 7365 4046 50  0000 L CNN
-F 1 "C" H 7365 3955 50  0000 L CNN
+F 1 ".001" H 7365 3955 50  0000 L CNN
 F 2 "" H 7288 3850 50  0001 C CNN
 F 3 "~" H 7250 4000 50  0001 C CNN

Commit message: Resistor enumeration
All resistors, diodes and transistors get numbers
Parts:
- gave numbers to parts that had none: 9
Changed lines of the file:
@@
 P 4500 3250
 AR Path="/62740CD0/627E8F93" Ref="R?"  Part="1"
-AR Path="/627D8A3A/627E8F93" Ref="R?"  Part="1"
-F 0 "R?" H 4570 3296 50  0000 L CNN
+AR Path="/627D8A3A/627E8F93" Ref="R59"  Part="1"
+F 0 "R59" H 4570 3296 50  0000 L CNN
 F 1 "1M" H 4570 3205 50  0000 L CNN
 F 2 "" V 4430 3250 50  0001 C CNN
@@
 P 5000 3750
 AR Path="/62740CD0/627E91C5" Ref="R?"  Part="1"
-AR Path="/627D8A3A/627E91C5" Ref="R?"  Part="1"
-F 0 "R?" H 5070 3796 50  0000 L CNN
+AR Path="/627D8A3A/627E91C5" Ref="R57"  Part="1"
+F 0 "R57" H 5070 3796 50  0000 L CNN
 F 1 "82k" H 5070 3705 50  0000 L CNN
 F 2 "" V 4930 3750 50  0001 C CNN
@@
 AR Path="/6276643A/627E95D6" Ref="Q?"  Part="1"
 AR Path="/62740CD0/627E95D6" Ref="Q?"  Part="1"
-AR Path="/627D8A3A/627E95D6" Ref="Q?"  Part="1"
-F 0 "Q?" H 5091 3046 50  0000 L CNN
+AR Path="/627D8A3A/627E95D6" Ref="Q12"  Part="1"
+F 0 "Q12" H 5091 3046 50  0000 L CNN
 F 1 "Q_NPN_BCE" H 5091 2955 50  0000 L CNN
 F 2 "" H 5100 3100 50  0001 C CNN
@@
 P 5250 4000
 AR Path="/62740CD0/627E9A1B" Ref="R?"  Part="1"
-AR Path="/627D8A3A/627E9A1B" Ref="R?"  Part="1"
-F 0 "R?" H 5320 4046 50  0000 L CNN
+AR Path="/627D8A3A/627E9A1B" Ref="R56"  Part="1"
+F 0 "R56" H 5320 4046 50  0000 L CNN
 F 1 "2.2M" H 5320 3955 50  0000 L CNN
 F 2 "" V 5180 4000 50  0001 C CNN
@@
 P 5500 4250
 AR Path="/62740CD0/627EA305" Ref="R?"  Part="1"
-AR Path="/627D8A3A/627EA305" Ref="R?"  Part="1"
-F 0 "R?" H 5570 4296 50  0000 L CNN
+AR Path="/627D8A3A/627EA305" Ref="R55"  Part="1"
+F 0 "R55" H 5570 4296 50  0000 L CNN
 F 1 "1M" H 5570 4205 50  0000 L CNN
 F 2 "" V 5430 4250 50  0001 C CNN
@@
 P 5500 3250
 AR Path="/62740CD0/627EAA10" Ref="R?"  Part="1"
-AR Path="/627D8A3A/627EAA10" Ref="R?"  Part="1"
-F 0 "R?" H 5570 3296 50  0000 L CNN
+AR Path="/627D8A3A/627EAA10" Ref="R54"  Part="1"
+F 0 "R54" H 5570 3296 50  0000 L CNN
 F 1 "10k" H 5570 3205 50  0000 L CNN
 F 2 "" V 5430 3250 50  0001 C CNN
@@
 AR Path="/6276643A/627EB49F" Ref="Q?"  Part="1"
 AR Path="/62740CD0/627EB49F" Ref="Q?"  Part="1"
-AR Path="/627D8A3A/627EB49F" Ref="Q?"  Part="1"
-F 0 "Q?" H 6091 4046 50  0000 L CNN
+AR Path="/627D8A3A/627EB49F" Ref="Q7"  Part="1"
+F 0 "Q7" H 6091 4046 50  0000 L CNN
 F 1 "Q_NPN_BCE" H 6091 3955 50  0000 L CNN
 F 2 "" H 6100 4100 50  0001 C CNN
@@
 $EndComp
 $Comp
-L Device:R R?
+L Device:R R52
 U 1 1 627F04C4
 P 6750 3500
-F 0 "R?" H 6820 3546 50  0000 L CNN
+F 0 "R52" H 6820 3546 50  0000 L CNN
 F 1 "10k" H 6820 3455 50  0000 L CNN
 F 2 "" V 6680 3500 50  0001 C CNN
@@
 $EndComp
 $Comp
-L Device:R R?
+L Device:R R53
 U 1 1 627F04CA
 P 6750 4000
-F 0 "R?" H 6820 4046 50  0000 L CNN
+F 0 "R53" H 6820 4046 50  0000 L CNN
 F 1 "47k" H 6820 3955 50  0000 L CNN
 F 2 "" V 6680 4000 50  0001 C CNN

Commit message: Footprints added
Added most of the footprints for a 0805 SMD PCB. some placeholder footprints added and some missing
Parts:
- C27, C28, C35, C36, C37, C38: renamed from C?; footprint (none) -> Capacitor_SMD:C_0805_2012Metric_Pad1.18x1.45mm_HandSolder
- Q12, Q7: footprint (none) -> Package_TO_SOT_SMD:SOT-23
- R52, R53, R54, R55, R56, R57, R59: footprint (none) -> Resistor_SMD:R_0805_2012Metric_Pad1.20x1.40mm_HandSolder
- gave numbers to parts that had none: 1
Changed lines of the file:
@@
 AR Path="/6276643A/627E8B98" Ref="C?"  Part="1"
 AR Path="/62740CD0/627E8B98" Ref="C?"  Part="1"
-AR Path="/627D8A3A/627E8B98" Ref="C?"  Part="1"
-F 0 "C?" H 4365 3046 50  0000 L CNN
+AR Path="/627D8A3A/627E8B98" Ref="C38"  Part="1"
+F 0 "C38" H 4365 3046 50  0000 L CNN
 F 1 ".047" H 4365 2955 50  0000 L CNN
-F 2 "" H 4288 2850 50  0001 C CNN
+F 2 "Capacitor_SMD:C_0805_2012Metric_Pad1.18x1.45mm_HandSolder" H 4288 2850 50  0001 C CNN
 F 3 "~" H 4250 3000 50  0001 C CNN
 	1    4250 3000
@@
 F 0 "R59" H 4570 3296 50  0000 L CNN
 F 1 "1M" H 4570 3205 50  0000 L CNN
-F 2 "" V 4430 3250 50  0001 C CNN
+F 2 "Resistor_SMD:R_0805_2012Metric_Pad1.20x1.40mm_HandSolder" V 4430 3250 50  0001 C CNN
 F 3 "~" H 4500 3250 50  0001 C CNN
 	1    4500 3250
@@
 F 0 "R57" H 5070 3796 50  0000 L CNN
 F 1 "82k" H 5070 3705 50  0000 L CNN
-F 2 "" V 4930 3750 50  0001 C CNN
+F 2 "Resistor_SMD:R_0805_2012Metric_Pad1.20x1.40mm_HandSolder" V 4930 3750 50  0001 C CNN
 F 3 "~" H 5000 3750 50  0001 C CNN
 	1    5000 3750
@@
 F 0 "Q12" H 5091 3046 50  0000 L CNN
 F 1 "Q_NPN_BCE" H 5091 2955 50  0000 L CNN
-F 2 "" H 5100 3100 50  0001 C CNN
+F 2 "Package_TO_SOT_SMD:SOT-23" H 5100 3100 50  0001 C CNN
 F 3 "~" H 4900 3000 50  0001 C CNN
 	1    4900 3000
@@
 F 0 "R56" H 5320 4046 50  0000 L CNN
 F 1 "2.2M" H 5320 3955 50  0000 L CNN
-F 2 "" V 5180 4000 50  0001 C CNN
+F 2 "Resistor_SMD:R_0805_2012Metric_Pad1.20x1.40mm_HandSolder" V 5180 4000 50  0001 C CNN
 F 3 "~" H 5250 4000 50  0001 C CNN
 	1    5250 4000
@@
 AR Path="/6276643A/627EA05F" Ref="C?"  Part="1"
 AR Path="/62740CD0/627EA05F" Ref="C?"  Part="1"
-AR Path="/627D8A3A/627EA05F" Ref="C?"  Part="1"
-F 0 "C?" H 5115 4296 50  0000 L CNN
+AR Path="/627D8A3A/627EA05F" Ref="C37"  Part="1"
+F 0 "C37" H 5115 4296 50  0000 L CNN
 F 1 ".018" H 5115 4205 50  0000 L CNN
-F 2 "" H 5038 4100 50  0001 C CNN
+F 2 "Capacitor_SMD:C_0805_2012Metric_Pad1.18x1.45mm_HandSolder" H 5038 4100 50  0001 C CNN
 F 3 "~" H 5000 4250 50  0001 C CNN
 	1    5000 4250
@@
 F 0 "R55" H 5570 4296 50  0000 L CNN
 F 1 "1M" H 5570 4205 50  0000 L CNN
-F 2 "" V 5430 4250 50  0001 C CNN
+F 2 "Resistor_SMD:R_0805_2012Metric_Pad1.20x1.40mm_HandSolder" V 5430 4250 50  0001 C CNN
 F 3 "~" H 5500 4250 50  0001 C CNN
 	1    5500 4250
@@
 F 0 "R54" H 5570 3296 50  0000 L CNN
 F 1 "10k" H 5570 3205 50  0000 L CNN
-F 2 "" V 5430 3250 50  0001 C CNN
+F 2 "Resistor_SMD:R_0805_2012Metric_Pad1.20x1.40mm_HandSolder" V 5430 3250 50  0001 C CNN
 F 3 "~" H 5500 3250 50  0001 C CNN
 	1    5500 3250
@@
 AR Path="/6276643A/627EADD0" Ref="C?"  Part="1"
 AR Path="/62740CD0/627EADD0" Ref="C?"  Part="1"
-AR Path="/627D8A3A/627EADD0" Ref="C?"  Part="1"
-F 0 "C?" H 5615 2796 50  0000 L CNN
+AR Path="/627D8A3A/627EADD0" Ref="C36"  Part="1"
+F 0 "C36" H 5615 2796 50  0000 L CNN
 F 1 ".001" H 5615 2705 50  0000 L CNN
-F 2 "" H 5538 2600 50  0001 C CNN
+F 2 "Capacitor_SMD:C_0805_2012Metric_Pad1.18x1.45mm_HandSolder" H 5538 2600 50  0001 C CNN
 F 3 "~" H 5500 2750 50  0001 C CNN
 	1    5500 2750
@@
 F 0 "Q7" H 6091 4046 50  0000 L CNN
 F 1 "Q_NPN_BCE" H 6091 3955 50  0000 L CNN
-F 2 "" H 6100 4100 50  0001 C CNN
+F 2 "Package_TO_SOT_SMD:SOT-23" H 6100 4100 50  0001 C CNN
 F 3 "~" H 5900 4000 50  0001 C CNN
 	1    5900 4000
@@
 $EndComp
 $Comp
-L Device:L L?
+L Device:L L1
 U 1 1 627EBD27
 P 6000 3250
-F 0 "L?" H 6053 3296 50  0000 L CNN
+F 0 "L1" H 6053 3296 50  0000 L CNN
 F 1 "45mH" H 6053 3205 50  0000 L CNN
 F 2 "" H 6000 3250 50  0001 C CNN
@@
 AR Path="/6276643A/627ECA20" Ref="C?"  Part="1"
 AR Path="/62740CD0/627ECA20" Ref="C?"  Part="1"
-AR Path="/627D8A3A/627ECA20" Ref="C?"  Part="1"
-F 0 "C?" H 6615 3296 50  0000 L CNN
+AR Path="/627D8A3A/627ECA20" Ref="C35"  Part="1"
+F 0 "C35" H 6615 3296 50  0000 L CNN
 F 1 ".0068" H 6615 3205 50  0000 L CNN
-F 2 "" H 6538 3100 50  0001 C CNN
+F 2 "Capacitor_SMD:C_0805_2012Metric_Pad1.18x1.45mm_HandSolder" H 6538 3100 50  0001 C CNN
 F 3 "~" H 6500 3250 50  0001 C CNN
 	1    6500 3250
@@
 F 0 "R52" H 6820 3546 50  0000 L CNN
 F 1 "10k" H 6820 3455 50  0000 L CNN
-F 2 "" V 6680 3500 50  0001 C CNN
+F 2 "Resistor_SMD:R_0805_2012Metric_Pad1.20x1.40mm_HandSolder" V 6680 3500 50  0001 C CNN
 F 3 "~" H 6750 3500 50  0001 C CNN
 	1    6750 3500
@@
 F 0 "R53" H 6820 4046 50  0000 L CNN
 F 1 "47k" H 6820 3955 50  0000 L CNN
-F 2 "" V 6680 4000 50  0001 C CNN
+F 2 "Resistor_SMD:R_0805_2012Metric_Pad1.20x1.40mm_HandSolder" V 6680 4000 50  0001 C CNN
 F 3 "~" H 6750 4000 50  0001 C CNN
 	1    6750 4000
@@
 AR Path="/6276643A/627F04D0" Ref="C?"  Part="1"
 AR Path="/62740CD0/627F04D0" Ref="C?"  Part="1"
-AR Path="/627D8A3A/627F04D0" Ref="C?"  Part="1"
-F 0 "C?" H 7365 3546 50  0000 L CNN
+AR Path="/627D8A3A/627F04D0" Ref="C27"  Part="1"
+F 0 "C27" H 7365 3546 50  0000 L CNN
 F 1 ".0022" H 7365 3455 50  0000 L CNN
-F 2 "" H 7288 3350 50  0001 C CNN
+F 2 "Capacitor_SMD:C_0805_2012Metric_Pad1.18x1.45mm_HandSolder" H 7288 3350 50  0001 C CNN
 F 3 "~" H 7250 3500 50  0001 C CNN
 	1    7250 3500
@@
 AR Path="/6276643A/627F04D6" Ref="C?"  Part="1"
 AR Path="/62740CD0/627F04D6" Ref="C?"  Part="1"
-AR Path="/627D8A3A/627F04D6" Ref="C?"  Part="1"
-F 0 "C?" H 7365 4046 50  0000 L CNN
+AR Path="/627D8A3A/627F04D6" Ref="C28"  Part="1"
+F 0 "C28" H 7365 4046 50  0000 L CNN
 F 1 ".001" H 7365 3955 50  0000 L CNN
-F 2 "" H 7288 3850 50  0001 C CNN
+F 2 "Capacitor_SMD:C_0805_2012Metric_Pad1.18x1.45mm_HandSolder" H 7288 3850 50  0001 C CNN
 F 3 "~" H 7250 4000 50  0001 C CNN
 	1    7250 4000
@@
 AR Path="/6276643A/627FCBB1" Ref="#PWR?"  Part="1"
 AR Path="/62740CD0/627FCBB1" Ref="#PWR?"  Part="1"
-AR Path="/627D8A3A/627FCBB1" Ref="#PWR?"  Part="1"
-F 0 "#PWR?" H 5000 2350 50  0001 C CNN
+AR Path="/627D8A3A/627FCBB1" Ref="#PWR0104"  Part="1"
+F 0 "#PWR0104" H 5000 2350 50  0001 C CNN
 F 1 "+6V" H 5015 2673 50  0000 C CNN
 F 2 "" H 5000 2500 50  0001 C CNN
@@
 AR Path="/6276643A/627FDAB6" Ref="#PWR?"  Part="1"
 AR Path="/62740CD0/627FDAB6" Ref="#PWR?"  Part="1"
-AR Path="/627D8A3A/627FDAB6" Ref="#PWR?"  Part="1"
-F 0 "#PWR?" H 6250 2850 50  0001 C CNN
+AR Path="/627D8A3A/627FDAB6" Ref="#PWR0105"  Part="1"
+F 0 "#PWR0105" H 6250 2850 50  0001 C CNN
 F 1 "+6V" H 6265 3173 50  0000 C CNN
 F 2 "" H 6250 3000 50  0001 C CNN
@@
 AR Path="/6276643A/627FF1DD" Ref="#PWR?"  Part="1"
 AR Path="/62740CD0/627FF1DD" Ref="#PWR?"  Part="1"
-AR Path="/627D8A3A/627FF1DD" Ref="#PWR?"  Part="1"
-F 0 "#PWR?" H 5000 4250 50  0001 C CNN
+AR Path="/627D8A3A/627FF1DD" Ref="#PWR0106"  Part="1"
+F 0 "#PWR0106" H 5000 4250 50  0001 C CNN
 F 1 "GND" H 5005 4327 50  0000 C CNN
 F 2 "" H 5000 4500 50  0001 C CNN
@@
 AR Path="/6276643A/627FF80A" Ref="#PWR?"  Part="1"
 AR Path="/62740CD0/627FF80A" Ref="#PWR?"  Part="1"
-AR Path="/627D8A3A/627FF80A" Ref="#PWR?"  Part="1"
-F 0 "#PWR?" H 5500 4250 50  0001 C CNN
+AR Path="/627D8A3A/627FF80A" Ref="#PWR0107"  Part="1"
+F 0 "#PWR0107" H 5500 4250 50  0001 C CNN
 F 1 "GND" H 5505 4327 50  0000 C CNN
 F 2 "" H 5500 4500 50  0001 C CNN
@@
 AR Path="/6276643A/628000B0" Ref="#PWR?"  Part="1"
 AR Path="/62740CD0/628000B0" Ref="#PWR?"  Part="1"
-AR Path="/627D8A3A/628000B0" Ref="#PWR?"  Part="1"
-F 0 "#PWR?" H 4500 3250 50  0001 C CNN
+AR Path="/627D8A3A/628000B0" Ref="#PWR0108"  Part="1"
+F 0 "#PWR0108" H 4500 3250 50  0001 C CNN
 F 1 "GND" H 4505 3327 50  0000 C CNN
 F 2 "" H 4500 3500 50  0001 C CNN
@@
 AR Path="/6276643A/62800C44" Ref="#PWR?"  Part="1"
 AR Path="/62740CD0/62800C44" Ref="#PWR?"  Part="1"
-AR Path="/627D8A3A/62800C44" Ref="#PWR?"  Part="1"
-F 0 "#PWR?" H 6000 4250 50  0001 C CNN
+AR Path="/627D8A3A/62800C44" Ref="#PWR0109"  Part="1"
+F 0 "#PWR0109" H 6000 4250 50  0001 C CNN
 F 1 "GND" H 6005 4327 50  0000 C CNN
 F 2 "" H 6000 4500 50  0001 C CNN

Commit message: SMD PCB
added all all Pcb layouts without CP footprint
Parts:
- L1: footprint (none) -> Connector_PinHeader_2.54mm:PinHeader_1x02_P2.54mm_Vertical
Changed lines of the file:
@@
 F 0 "L1" H 6053 3296 50  0000 L CNN
 F 1 "45mH" H 6053 3205 50  0000 L CNN
-F 2 "" H 6000 3250 50  0001 C CNN
+F 2 "Connector_PinHeader_2.54mm:PinHeader_1x02_P2.54mm_Vertical" H 6000 3250 50  0001 C CNN
 F 3 "~" H 6000 3250 50  0001 C CNN
 	1    6000 3250

Commit message: changed some stuff
Parts:
- C27, C28, C35, C36, C37, C38: footprint Capacitor_SMD:C_0805_2012Metric_Pad1.18x1.45mm_HandSolder -> Capacitor_SMD:C_0805_2012Metric
- Q12, Q7: footprint Package_TO_SOT_SMD:SOT-23 -> Package_TO_SOT_SMD:SOT-89-3
- R52, R53, R54, R55, R56, R57, R59: footprint Resistor_SMD:R_0805_2012Metric_Pad1.20x1.40mm_HandSolder -> Resistor_SMD:R_0805_2012Metric
Changed lines of the file:
@@
 $Descr A4 11693 8268
 encoding utf-8
-Sheet 2 7
+Sheet 2 8
 Title ""
 Date ""
@@
 F 0 "C38" H 4365 3046 50  0000 L CNN
 F 1 ".047" H 4365 2955 50  0000 L CNN
-F 2 "Capacitor_SMD:C_0805_2012Metric_Pad1.18x1.45mm_HandSolder" H 4288 2850 50  0001 C CNN
+F 2 "Capacitor_SMD:C_0805_2012Metric" H 4288 2850 50  0001 C CNN
 F 3 "~" H 4250 3000 50  0001 C CNN
 	1    4250 3000
@@
 F 0 "R59" H 4570 3296 50  0000 L CNN
 F 1 "1M" H 4570 3205 50  0000 L CNN
-F 2 "Resistor_SMD:R_0805_2012Metric_Pad1.20x1.40mm_HandSolder" V 4430 3250 50  0001 C CNN
+F 2 "Resistor_SMD:R_0805_2012Metric" V 4430 3250 50  0001 C CNN
 F 3 "~" H 4500 3250 50  0001 C CNN
 	1    4500 3250
@@
 F 0 "R57" H 5070 3796 50  0000 L CNN
 F 1 "82k" H 5070 3705 50  0000 L CNN
-F 2 "Resistor_SMD:R_0805_2012Metric_Pad1.20x1.40mm_HandSolder" V 4930 3750 50  0001 C CNN
+F 2 "Resistor_SMD:R_0805_2012Metric" V 4930 3750 50  0001 C CNN
 F 3 "~" H 5000 3750 50  0001 C CNN
 	1    5000 3750
@@
 F 0 "Q12" H 5091 3046 50  0000 L CNN
 F 1 "Q_NPN_BCE" H 5091 2955 50  0000 L CNN
-F 2 "Package_TO_SOT_SMD:SOT-23" H 5100 3100 50  0001 C CNN
+F 2 "Package_TO_SOT_SMD:SOT-89-3" H 5100 3100 50  0001 C CNN
 F 3 "~" H 4900 3000 50  0001 C CNN
 	1    4900 3000
@@
 F 0 "R56" H 5320 4046 50  0000 L CNN
 F 1 "2.2M" H 5320 3955 50  0000 L CNN
-F 2 "Resistor_SMD:R_0805_2012Metric_Pad1.20x1.40mm_HandSolder" V 5180 4000 50  0001 C CNN
+F 2 "Resistor_SMD:R_0805_2012Metric" V 5180 4000 50  0001 C CNN
 F 3 "~" H 5250 4000 50  0001 C CNN
 	1    5250 4000
@@
 F 0 "C37" H 5115 4296 50  0000 L CNN
 F 1 ".018" H 5115 4205 50  0000 L CNN
-F 2 "Capacitor_SMD:C_0805_2012Metric_Pad1.18x1.45mm_HandSolder" H 5038 4100 50  0001 C CNN
+F 2 "Capacitor_SMD:C_0805_2012Metric" H 5038 4100 50  0001 C CNN
 F 3 "~" H 5000 4250 50  0001 C CNN
 	1    5000 4250
@@
 F 0 "R55" H 5570 4296 50  0000 L CNN
 F 1 "1M" H 5570 4205 50  0000 L CNN
-F 2 "Resistor_SMD:R_0805_2012Metric_Pad1.20x1.40mm_HandSolder" V 5430 4250 50  0001 C CNN
+F 2 "Resistor_SMD:R_0805_2012Metric" V 5430 4250 50  0001 C CNN
 F 3 "~" H 5500 4250 50  0001 C CNN
 	1    5500 4250
@@
 F 0 "R54" H 5570 3296 50  0000 L CNN
 F 1 "10k" H 5570 3205 50  0000 L CNN
-F 2 "Resistor_SMD:R_0805_2012Metric_Pad1.20x1.40mm_HandSolder" V 5430 3250 50  0001 C CNN
+F 2 "Resistor_SMD:R_0805_2012Metric" V 5430 3250 50  0001 C CNN
 F 3 "~" H 5500 3250 50  0001 C CNN
 	1    5500 3250
@@
 F 0 "C36" H 5615 2796 50  0000 L CNN
 F 1 ".001" H 5615 2705 50  0000 L CNN
-F 2 "Capacitor_SMD:C_0805_2012Metric_Pad1.18x1.45mm_HandSolder" H 5538 2600 50  0001 C CNN
+F 2 "Capacitor_SMD:C_0805_2012Metric" H 5538 2600 50  0001 C CNN
 F 3 "~" H 5500 2750 50  0001 C CNN
 	1    5500 2750
@@
 F 0 "Q7" H 6091 4046 50  0000 L CNN
 F 1 "Q_NPN_BCE" H 6091 3955 50  0000 L CNN
-F 2 "Package_TO_SOT_SMD:SOT-23" H 6100 4100 50  0001 C CNN
+F 2 "Package_TO_SOT_SMD:SOT-89-3" H 6100 4100 50  0001 C CNN
 F 3 "~" H 5900 4000 50  0001 C CNN
 	1    5900 4000
@@
 F 0 "C35" H 6615 3296 50  0000 L CNN
 F 1 ".0068" H 6615 3205 50  0000 L CNN
-F 2 "Capacitor_SMD:C_0805_2012Metric_Pad1.18x1.45mm_HandSolder" H 6538 3100 50  0001 C CNN
+F 2 "Capacitor_SMD:C_0805_2012Metric" H 6538 3100 50  0001 C CNN
 F 3 "~" H 6500 3250 50  0001 C CNN
 	1    6500 3250
@@
 F 0 "R52" H 6820 3546 50  0000 L CNN
 F 1 "10k" H 6820 3455 50  0000 L CNN
-F 2 "Resistor_SMD:R_0805_2012Metric_Pad1.20x1.40mm_HandSolder" V 6680 3500 50  0001 C CNN
+F 2 "Resistor_SMD:R_0805_2012Metric" V 6680 3500 50  0001 C CNN
 F 3 "~" H 6750 3500 50  0001 C CNN
 	1    6750 3500
@@
 F 0 "R53" H 6820 4046 50  0000 L CNN
 F 1 "47k" H 6820 3955 50  0000 L CNN
-F 2 "Resistor_SMD:R_0805_2012Metric_Pad1.20x1.40mm_HandSolder" V 6680 4000 50  0001 C CNN
+F 2 "Resistor_SMD:R_0805_2012Metric" V 6680 4000 50  0001 C CNN
 F 3 "~" H 6750 4000 50  0001 C CNN
 	1    6750 4000
@@
 F 0 "C27" H 7365 3546 50  0000 L CNN
 F 1 ".0022" H 7365 3455 50  0000 L CNN
-F 2 "Capacitor_SMD:C_0805_2012Metric_Pad1.18x1.45mm_HandSolder" H 7288 3350 50  0001 C CNN
+F 2 "Capacitor_SMD:C_0805_2012Metric" H 7288 3350 50  0001 C CNN
 F 3 "~" H 7250 3500 50  0001 C CNN
 	1    7250 3500
@@
 F 0 "C28" H 7365 4046 50  0000 L CNN
 F 1 ".001" H 7365 3955 50  0000 L CNN
-F 2 "Capacitor_SMD:C_0805_2012Metric_Pad1.18x1.45mm_HandSolder" H 7288 3850 50  0001 C CNN
+F 2 "Capacitor_SMD:C_0805_2012Metric" H 7288 3850 50  0001 C CNN
 F 3 "~" H 7250 4000 50  0001 C CNN
 	1    7250 4000
