File: DR-55-Kick/DR-55-Kick.sch (KiCad schematic (older format))
At the start: 19 parts, among them Q1 Q_NPN_BCE, Q2 Q_NPN_BCE

Commit message: changed some stuff
Parts:
- C1, C2, C3, C4, C5, C?26: footprint Capacitor_SMD:C_0805_2012Metric_Pad1.18x1.45mm_HandSolder -> Capacitor_SMD:C_0805_2012Metric
- Q1, Q2: footprint Package_TO_SOT_SMD:SOT-23 -> Package_TO_SOT_SMD:SOT-89-3
- R1, R10, R11, R12, R2, R4, R5, R6, R7, R8, R9: footprint Resistor_SMD:R_0805_2012Metric_Pad1.20x1.40mm_HandSolder -> Resistor_SMD:R_0805_2012Metric
Changed lines of the file:
@@
 $Descr A4 11693 8268
 encoding utf-8
-Sheet 5 7
+Sheet 5 8
 Title ""
 Date ""
@@
 F 0 "R11" V 2043 1500 50  0000 C CNN
 F 1 "680k" V 2134 1500 50  0000 C CNN
-F 2 "Resistor_SMD:R_0805_2012Metric_Pad1.20x1.40mm_HandSolder" V 2180 1500 50  0001 C CNN
+F 2 "Resistor_SMD:R_0805_2012Metric" V 2180 1500 50  0001 C CNN
 F 3 "~" H 2250 1500 50  0001 C CNN
 	1    2250 1500
@@
 F 0 "C5" H 2615 2046 50  0000 L CNN
 F 1 ".068" H 2615 1955 50  0000 L CNN
-F 2 "Capacitor_SMD:C_0805_2012Metric_Pad1.18x1.45mm_HandSolder" H 2538 1850 50  0001 C CNN
+F 2 "Capacitor_SMD:C_0805_2012Metric" H 2538 1850 50  0001 C CNN
 F 3 "~" H 2500 2000 50  0001 C CNN
 	1    2500 2000
@@
 F 0 "Q2" H 4091 2546 50  0000 L CNN
 F 1 "Q_NPN_BCE" H 4091 2455 50  0000 L CNN
-F 2 "Package_TO_SOT_SMD:SOT-23" H 4100 2600 50  0001 C CNN
+F 2 "Package_TO_SOT_SMD:SOT-89-3" H 4100 2600 50  0001 C CNN
 F 3 "~" H 3900 2500 50  0001 C CNN
 	1    3900 2500
@@
 F 0 "C4" H 2365 2546 50  0000 L CNN
 F 1 ".068" H 2365 2455 50  0000 L CNN
-F 2 "Capacitor_SMD:C_0805_2012Metric_Pad1.18x1.45mm_HandSolder" H 2288 2350 50  0001 C CNN
+F 2 "Capacitor_SMD:C_0805_2012Metric" H 2288 2350 50  0001 C CNN
 F 3 "~" H 2250 2500 50  0001 C CNN
 	1    2250 2500
@@
 F 0 "C3" H 2865 2546 50  0000 L CNN
 F 1 ".068" H 2865 2455 50  0000 L CNN
-F 2 "Capacitor_SMD:C_0805_2012Metric_Pad1.18x1.45mm_HandSolder" H 2788 2350 50  0001 C CNN
+F 2 "Capacitor_SMD:C_0805_2012Metric" H 2788 2350 50  0001 C CNN
 F 3 "~" H 2750 2500 50  0001 C CNN
 	1    2750 2500
@@
 F 0 "R9" V 1793 2750 50  0000 C CNN
 F 1 "22k" V 1884 2750 50  0000 C CNN
-F 2 "Resistor_SMD:R_0805_2012Metric_Pad1.20x1.40mm_HandSolder" V 1930 2750 50  0001 C CNN
+F 2 "Resistor_SMD:R_0805_2012Metric" V 1930 2750 50  0001 C CNN
 F 3 "~" H 2000 2750 50  0001 C CNN
 	1    2000 2750
@@
 F 0 "R8" V 2293 2750 50  0000 C CNN
 F 1 "22k" V 2384 2750 50  0000 C CNN
-F 2 "Resistor_SMD:R_0805_2012Metric_Pad1.20x1.40mm_HandSolder" V 2430 2750 50  0001 C CNN
+F 2 "Resistor_SMD:R_0805_2012Metric" V 2430 2750 50  0001 C CNN
 F 3 "~" H 2500 2750 50  0001 C CNN
 	1    2500 2750
@@
 F 0 "R7" V 2793 2750 50  0000 C CNN
 F 1 "22k" V 2884 2750 50  0000 C CNN
-F 2 "Resistor_SMD:R_0805_2012Metric_Pad1.20x1.40mm_HandSolder" V 2930 2750 50  0001 C CNN
+F 2 "Resistor_SMD:R_0805_2012Metric" V 2930 2750 50  0001 C CNN
 F 3 "~" H 3000 2750 50  0001 C CNN
 	1    3000 2750
@@
 F 0 "C2" H 3365 2546 50  0000 L CNN
 F 1 ".068" H 3365 2455 50  0000 L CNN
-F 2 "Capacitor_SMD:C_0805_2012Metric_Pad1.18x1.45mm_HandSolder" H 3288 2350 50  0001 C CNN
+F 2 "Capacitor_SMD:C_0805_2012Metric" H 3288 2350 50  0001 C CNN
 F 3 "~" H 3250 2500 50  0001 C CNN
 	1    3250 2500
@@
 F 0 "R5" V 3293 2250 50  0000 C CNN
 F 1 "2.2M" V 3384 2250 50  0000 C CNN
-F 2 "Resistor_SMD:R_0805_2012Metric_Pad1.20x1.40mm_HandSolder" V 3430 2250 50  0001 C CNN
+F 2 "Resistor_SMD:R_0805_2012Metric" V 3430 2250 50  0001 C CNN
 F 3 "~" H 3500 2250 50  0001 C CNN
 	1    3500 2250
@@
 F 0 "R4" V 3793 1750 50  0000 C CNN
 F 1 "10k" V 3884 1750 50  0000 C CNN
-F 2 "Resistor_SMD:R_0805_2012Metric_Pad1.20x1.40mm_HandSolder" V 3930 1750 50  0001 C CNN
+F 2 "Resistor_SMD:R_0805_2012Metric" V 3930 1750 50  0001 C CNN
 F 3 "~" H 4000 1750 50  0001 C CNN
 	1    4000 1750
@@
 F 0 "C1" H 4865 2546 50  0000 L CNN
 F 1 ".047" H 4865 2455 50  0000 L CNN
-F 2 "Capacitor_SMD:C_0805_2012Metric_Pad1.18x1.45mm_HandSolder" H 4788 2350 50  0001 C CNN
+F 2 "Capacitor_SMD:C_0805_2012Metric" H 4788 2350 50  0001 C CNN
 F 3 "~" H 4750 2500 50  0001 C CNN
 	1    4750 2500
@@
 F 0 "R2" V 4793 2250 50  0000 C CNN
 F 1 "220k" V 4884 2250 50  0000 C CNN
-F 2 "Resistor_SMD:R_0805_2012Metric_Pad1.20x1.40mm_HandSolder" V 4930 2250 50  0001 C CNN
+F 2 "Resistor_SMD:R_0805_2012Metric" V 4930 2250 50  0001 C CNN
 F 3 "~" H 5000 2250 50  0001 C CNN
 	1    5000 2250
@@
 F 0 "Q1" H 5591 2546 50  0000 L CNN
 F 1 "Q_NPN_BCE" H 5591 2455 50  0000 L CNN
-F 2 "Package_TO_SOT_SMD:SOT-23" H 5600 2600 50  0001 C CNN
+F 2 "Package_TO_SOT_SMD:SOT-89-3" H 5600 2600 50  0001 C CNN
 F 3 "~" H 5400 2500 50  0001 C CNN
 	1    5400 2500
@@
 F 0 "R1" V 5293 3250 50  0000 C CNN
 F 1 "1k" V 5384 3250 50  0000 C CNN
-F 2 "Resistor_SMD:R_0805_2012Metric_Pad1.20x1.40mm_HandSolder" V 5430 3250 50  0001 C CNN
+F 2 "Resistor_SMD:R_0805_2012Metric" V 5430 3250 50  0001 C CNN
 F 3 "~" H 5500 3250 50  0001 C CNN
 	1    5500 3250
@@
 F 0 "R6" V 5293 1750 50  0000 C CNN
 F 1 "22k" V 5384 1750 50  0000 C CNN
-F 2 "Resistor_SMD:R_0805_2012Metric_Pad1.20x1.40mm_HandSolder" V 5430 1750 50  0001 C CNN
+F 2 "Resistor_SMD:R_0805_2012Metric" V 5430 1750 50  0001 C CNN
 F 3 "~" H 5500 1750 50  0001 C CNN
 	1    5500 1750
@@
 F 0 "R10" V 5793 2250 50  0000 C CNN
 F 1 "150k" V 5884 2250 50  0000 C CNN
-F 2 "Resistor_SMD:R_0805_2012Metric_Pad1.20x1.40mm_HandSolder" V 5930 2250 50  0001 C CNN
+F 2 "Resistor_SMD:R_0805_2012Metric" V 5930 2250 50  0001 C CNN
 F 3 "~" H 6000 2250 50  0001 C CNN
 	1    6000 2250
@@
 F 0 "C?26" H 6115 2796 50  0000 L CNN
 F 1 ".027" H 6115 2705 50  0000 L CNN
-F 2 "Capacitor_SMD:C_0805_2012Metric_Pad1.18x1.45mm_HandSolder" H 6038 2600 50  0001 C CNN
+F 2 "Capacitor_SMD:C_0805_2012Metric" H 6038 2600 50  0001 C CNN
 F 3 "~" H 6000 2750 50  0001 C CNN
 	1    6000 2750
@@
 F 0 "R12" V 3793 3250 50  0000 C CNN
 F 1 "820" V 3884 3250 50  0000 C CNN
-F 2 "Resistor_SMD:R_0805_2012Metric_Pad1.20x1.40mm_HandSolder" V 3930 3250 50  0001 C CNN
+F 2 "Resistor_SMD:R_0805_2012Metric" V 3930 3250 50  0001 C CNN
 F 3 "~" H 4000 3250 50  0001 C CNN
 	1    4000 3250
