File: DR-55-Noise/DR-55-Noise.sch (KiCad schematic (older format))
At the start: 9 parts

Commit message: Values
Added Values to all components
Parts:
- C?: value C -> .0022
- C?: value CP -> 22/10
- R? (x2): value R -> 2.2M
- R?: value R -> 10k
- R?: value R -> 1K
- RV?: value R_POT_TRIM -> 10kB
Changed lines of the file:
@@
 $Descr A4 11693 8268
 encoding utf-8
-Sheet 5 7
+Sheet 4 7
 Title ""
 Date ""
@@
 AR Path="/62804B1F/6283DABC" Ref="C?"  Part="1"
 F 0 "C?" H 6365 5046 50  0000 L CNN
-F 1 "C" H 6365 4955 50  0000 L CNN
+F 1 ".0022" H 6365 4955 50  0000 L CNN
 F 2 "" H 6288 4850 50  0001 C CNN
 F 3 "~" H 6250 5000 50  0001 C CNN
@@
 AR Path="/62804B1F/628482E9" Ref="R?"  Part="1"
 F 0 "R?" H 6570 4796 50  0000 L CNN
-F 1 "R" H 6570 4705 50  0000 L CNN
+F 1 "2.2M" H 6570 4705 50  0000 L CNN
 F 2 "" V 6430 4750 50  0001 C CNN
 F 3 "~" H 6500 4750 50  0001 C CNN
@@
 AR Path="/62804B1F/62848B5C" Ref="R?"  Part="1"
 F 0 "R?" H 5070 4796 50  0000 L CNN
-F 1 "R" H 5070 4705 50  0000 L CNN
+F 1 "2.2M" H 5070 4705 50  0000 L CNN
 F 2 "" V 4930 4750 50  0001 C CNN
 F 3 "~" H 5000 4750 50  0001 C CNN
@@
 AR Path="/62804B1F/6284AA04" Ref="R?"  Part="1"
 F 0 "R?" H 6320 4046 50  0000 L CNN
-F 1 "R" H 6320 3955 50  0000 L CNN
+F 1 "10k" H 6320 3955 50  0000 L CNN
 F 2 "" V 6180 4000 50  0001 C CNN
 F 3 "~" H 6250 4000 50  0001 C CNN
@@
 AR Path="/62804B1F/6284C368" Ref="R?"  Part="1"
 F 0 "R?" H 8320 4046 50  0000 L CNN
-F 1 "R" H 8320 3955 50  0000 L CNN
+F 1 "1K" H 8320 3955 50  0000 L CNN
 F 2 "" V 8180 4000 50  0001 C CNN
 F 3 "~" H 8250 4000 50  0001 C CNN
@@
 P 8000 4750
 F 0 "C?" H 8118 4796 50  0000 L CNN
-F 1 "CP" H 8118 4705 50  0000 L CNN
+F 1 "22/10" H 8118 4705 50  0000 L CNN
 F 2 "" H 8038 4600 50  0001 C CNN
 F 3 "~" H 8000 4750 50  0001 C CNN
@@
 P 7000 4250
 F 0 "RV?" H 6930 4296 50  0000 R CNN
-F 1 "R_POT_TRIM" H 6930 4205 50  0000 R CNN
+F 1 "10kB" H 6930 4205 50  0000 R CNN
 F 2 "" H 7000 4250 50  0001 C CNN
 F 3 "~" H 7000 4250 50  0001 C CNN

Commit message: Resistor enumeration
All resistors, diodes and transistors get numbers
Parts:
- gave numbers to parts that had none: 7
Changed lines of the file:
@@
 AR Path="/62740CD0/6283DAD4" Ref="Q?"  Part="1"
 AR Path="/62804339/6283DAD4" Ref="Q?"  Part="1"
-AR Path="/62804B1F/6283DAD4" Ref="Q?"  Part="1"
-F 0 "Q?" H 5591 5046 50  0000 L CNN
+AR Path="/62804B1F/6283DAD4" Ref="Q8"  Part="1"
+F 0 "Q8" H 5591 5046 50  0000 L CNN
 F 1 "Q_NPN_BCE" H 5591 4955 50  0000 L CNN
 F 2 "" H 5600 5100 50  0001 C CNN
@@
 AR Path="/62740CD0/628480A0" Ref="Q?"  Part="1"
 AR Path="/62804339/628480A0" Ref="Q?"  Part="1"
-AR Path="/62804B1F/628480A0" Ref="Q?"  Part="1"
-F 0 "Q?" H 7091 5046 50  0000 L CNN
+AR Path="/62804B1F/628480A0" Ref="Q9"  Part="1"
+F 0 "Q9" H 7091 5046 50  0000 L CNN
 F 1 "Q_NPN_BCE" H 7091 4955 50  0000 L CNN
 F 2 "" H 7100 5100 50  0001 C CNN
@@
 AR Path="/62740CD0/628482E9" Ref="R?"  Part="1"
 AR Path="/62804339/628482E9" Ref="R?"  Part="1"
-AR Path="/62804B1F/628482E9" Ref="R?"  Part="1"
-F 0 "R?" H 6570 4796 50  0000 L CNN
+AR Path="/62804B1F/628482E9" Ref="R51"  Part="1"
+F 0 "R51" H 6570 4796 50  0000 L CNN
 F 1 "2.2M" H 6570 4705 50  0000 L CNN
 F 2 "" V 6430 4750 50  0001 C CNN
@@
 AR Path="/62740CD0/62848B5C" Ref="R?"  Part="1"
 AR Path="/62804339/62848B5C" Ref="R?"  Part="1"
-AR Path="/62804B1F/62848B5C" Ref="R?"  Part="1"
-F 0 "R?" H 5070 4796 50  0000 L CNN
+AR Path="/62804B1F/62848B5C" Ref="R50"  Part="1"
+F 0 "R50" H 5070 4796 50  0000 L CNN
 F 1 "2.2M" H 5070 4705 50  0000 L CNN
 F 2 "" V 4930 4750 50  0001 C CNN
@@
 AR Path="/62740CD0/6284AA04" Ref="R?"  Part="1"
 AR Path="/62804339/6284AA04" Ref="R?"  Part="1"
-AR Path="/62804B1F/6284AA04" Ref="R?"  Part="1"
-F 0 "R?" H 6320 4046 50  0000 L CNN
+AR Path="/62804B1F/6284AA04" Ref="R49"  Part="1"
+F 0 "R49" H 6320 4046 50  0000 L CNN
 F 1 "10k" H 6320 3955 50  0000 L CNN
 F 2 "" V 6180 4000 50  0001 C CNN
@@
 AR Path="/62740CD0/6284C368" Ref="R?"  Part="1"
 AR Path="/62804339/6284C368" Ref="R?"  Part="1"
-AR Path="/62804B1F/6284C368" Ref="R?"  Part="1"
-F 0 "R?" H 8320 4046 50  0000 L CNN
+AR Path="/62804B1F/6284C368" Ref="R24"  Part="1"
+F 0 "R24" H 8320 4046 50  0000 L CNN
 F 1 "1K" H 8320 3955 50  0000 L CNN
 F 2 "" V 8180 4000 50  0001 C CNN
@@
 	8000 5500 8000 4900
 $Comp
-L Device:R_POT_TRIM RV?
+L Device:R_POT_TRIM VR7
 U 1 1 628539C9
 P 7000 4250
-F 0 "RV?" H 6930 4296 50  0000 R CNN
+F 0 "VR7" H 6930 4296 50  0000 R CNN
 F 1 "10kB" H 6930 4205 50  0000 R CNN
 F 2 "" H 7000 4250 50  0001 C CNN

Commit message: Footprints added
Added most of the footprints for a 0805 SMD PCB. some placeholder footprints added and some missing
Parts:
- C34: renamed from C?; footprint (none) -> Capacitor_SMD:C_0805_2012Metric_Pad1.18x1.45mm_HandSolder
- Q8, Q9: footprint (none) -> Package_TO_SOT_SMD:SOT-23
- R24, R49, R50, R51: footprint (none) -> Resistor_SMD:R_0805_2012Metric_Pad1.20x1.40mm_HandSolder
- gave numbers to parts that had none: 1
Changed lines of the file:
@@
 AR Path="/62740CD0/6283DA72" Ref="#PWR?"  Part="1"
 AR Path="/62804339/6283DA72" Ref="#PWR?"  Part="1"
-AR Path="/62804B1F/6283DA72" Ref="#PWR?"  Part="1"
-F 0 "#PWR?" H 8500 3350 50  0001 C CNN
+AR Path="/62804B1F/6283DA72" Ref="#PWR0117"  Part="1"
+F 0 "#PWR0117" H 8500 3350 50  0001 C CNN
 F 1 "+6V" H 8515 3673 50  0000 C CNN
 F 2 "" H 8500 3500 50  0001 C CNN
@@
 AR Path="/62740CD0/6283DABC" Ref="C?"  Part="1"
 AR Path="/62804339/6283DABC" Ref="C?"  Part="1"
-AR Path="/62804B1F/6283DABC" Ref="C?"  Part="1"
-F 0 "C?" H 6365 5046 50  0000 L CNN
+AR Path="/62804B1F/6283DABC" Ref="C34"  Part="1"
+F 0 "C34" H 6365 5046 50  0000 L CNN
 F 1 ".0022" H 6365 4955 50  0000 L CNN
-F 2 "" H 6288 4850 50  0001 C CNN
+F 2 "Capacitor_SMD:C_0805_2012Metric_Pad1.18x1.45mm_HandSolder" H 6288 4850 50  0001 C CNN
 F 3 "~" H 6250 5000 50  0001 C CNN
 	1    6250 5000
@@
 F 0 "Q8" H 5591 5046 50  0000 L CNN
 F 1 "Q_NPN_BCE" H 5591 4955 50  0000 L CNN
-F 2 "" H 5600 5100 50  0001 C CNN
+F 2 "Package_TO_SOT_SMD:SOT-23" H 5600 5100 50  0001 C CNN
 F 3 "~" H 5400 5000 50  0001 C CNN
 	1    5400 5000
@@
 AR Path="/62740CD0/6283DB16" Ref="#PWR?"  Part="1"
 AR Path="/62804339/6283DB16" Ref="#PWR?"  Part="1"
-AR Path="/62804B1F/6283DB16" Ref="#PWR?"  Part="1"
-F 0 "#PWR?" H 7000 5250 50  0001 C CNN
+AR Path="/62804B1F/6283DB16" Ref="#PWR0118"  Part="1"
+F 0 "#PWR0118" H 7000 5250 50  0001 C CNN
 F 1 "GND" H 7005 5327 50  0000 C CNN
 F 2 "" H 7000 5500 50  0001 C CNN
@@
 F 0 "Q9" H 7091 5046 50  0000 L CNN
 F 1 "Q_NPN_BCE" H 7091 4955 50  0000 L CNN
-F 2 "" H 7100 5100 50  0001 C CNN
+F 2 "Package_TO_SOT_SMD:SOT-23" H 7100 5100 50  0001 C CNN
 F 3 "~" H 6900 5000 50  0001 C CNN
 	1    6900 5000
@@
 F 0 "R51" H 6570 4796 50  0000 L CNN
 F 1 "2.2M" H 6570 4705 50  0000 L CNN
-F 2 "" V 6430 4750 50  0001 C CNN
+F 2 "Resistor_SMD:R_0805_2012Metric_Pad1.20x1.40mm_HandSolder" V 6430 4750 50  0001 C CNN
 F 3 "~" H 6500 4750 50  0001 C CNN
 	1    6500 4750
@@
 F 0 "R50" H 5070 4796 50  0000 L CNN
 F 1 "2.2M" H 5070 4705 50  0000 L CNN
-F 2 "" V 4930 4750 50  0001 C CNN
+F 2 "Resistor_SMD:R_0805_2012Metric_Pad1.20x1.40mm_HandSolder" V 4930 4750 50  0001 C CNN
 F 3 "~" H 5000 4750 50  0001 C CNN
 	1    5000 4750
@@
 F 0 "R49" H 6320 4046 50  0000 L CNN
 F 1 "10k" H 6320 3955 50  0000 L CNN
-F 2 "" V 6180 4000 50  0001 C CNN
+F 2 "Resistor_SMD:R_0805_2012Metric_Pad1.20x1.40mm_HandSolder" V 6180 4000 50  0001 C CNN
 F 3 "~" H 6250 4000 50  0001 C CNN
 	1    6250 4000
@@
 F 0 "R24" H 8320 4046 50  0000 L CNN
 F 1 "1K" H 8320 3955 50  0000 L CNN
-F 2 "" V 8180 4000 50  0001 C CNN
+F 2 "Resistor_SMD:R_0805_2012Metric_Pad1.20x1.40mm_HandSolder" V 8180 4000 50  0001 C CNN
 F 3 "~" H 8250 4000 50  0001 C CNN
 	1    8250 4000
@@
 AR Path="/62740CD0/6284EF72" Ref="#PWR?"  Part="1"
 AR Path="/62804339/6284EF72" Ref="#PWR?"  Part="1"
-AR Path="/62804B1F/6284EF72" Ref="#PWR?"  Part="1"
-F 0 "#PWR?" H 5500 5250 50  0001 C CNN
+AR Path="/62804B1F/6284EF72" Ref="#PWR0119"  Part="1"
+F 0 "#PWR0119" H 5500 5250 50  0001 C CNN
 F 1 "GND" H 5505 5327 50  0000 C CNN
 F 2 "" H 5500 5500 50  0001 C CNN
@@
 AR Path="/62740CD0/6284F987" Ref="#PWR?"  Part="1"
 AR Path="/62804339/6284F987" Ref="#PWR?"  Part="1"
-AR Path="/62804B1F/6284F987" Ref="#PWR?"  Part="1"
-F 0 "#PWR?" H 8000 5250 50  0001 C CNN
+AR Path="/62804B1F/6284F987" Ref="#PWR0120"  Part="1"
+F 0 "#PWR0120" H 8000 5250 50  0001 C CNN
 F 1 "GND" H 8005 5327 50  0000 C CNN
 F 2 "" H 8000 5500 50  0001 C CNN
@@
 	7000 5200 7000 5500
 $Comp
-L Device:CP C?
+L Device:CP C14
 U 1 1 6285189A
 P 8000 4750
-F 0 "C?" H 8118 4796 50  0000 L CNN
+F 0 "C14" H 8118 4796 50  0000 L CNN
 F 1 "22/10" H 8118 4705 50  0000 L CNN
 F 2 "" H 8038 4600 50  0001 C CNN

Commit message: SMD PCB
added all all Pcb layouts without CP footprint
Parts:
- C14: footprint (none) -> Connector_PinHeader_2.54mm:PinHeader_1x02_P2.54mm_Vertical
- VR7: footprint (none) -> Connector_PinHeader_2.54mm:PinHeader_1x03_P2.54mm_Vertical
Changed lines of the file:
@@
 F 0 "C14" H 8118 4796 50  0000 L CNN
 F 1 "22/10" H 8118 4705 50  0000 L CNN
-F 2 "" H 8038 4600 50  0001 C CNN
+F 2 "Connector_PinHeader_2.54mm:PinHeader_1x02_P2.54mm_Vertical" H 8038 4600 50  0001 C CNN
 F 3 "~" H 8000 4750 50  0001 C CNN
 	1    8000 4750
@@
 F 0 "VR7" H 6930 4296 50  0000 R CNN
 F 1 "10kB" H 6930 4205 50  0000 R CNN
-F 2 "" H 7000 4250 50  0001 C CNN
+F 2 "Connector_PinHeader_2.54mm:PinHeader_1x03_P2.54mm_Vertical" H 7000 4250 50  0001 C CNN
 F 3 "~" H 7000 4250 50  0001 C CNN
 	1    7000 4250

Commit message: changed some stuff
Parts:
- C14: footprint Connector_PinHeader_2.54mm:PinHeader_1x02_P2.54mm_Vertical -> Capacitor_THT:CP_Radial_D5.0mm_P2.50mm
- C34: footprint Capacitor_SMD:C_0805_2012Metric_Pad1.18x1.45mm_HandSolder -> Capacitor_SMD:C_0805_2012Metric
- Q8, Q9: footprint Package_TO_SOT_SMD:SOT-23 -> Package_TO_SOT_SMD:SOT-89-3
- R24, R49, R50, R51: footprint Resistor_SMD:R_0805_2012Metric_Pad1.20x1.40mm_HandSolder -> Resistor_SMD:R_0805_2012Metric
- VR7: footprint Connector_PinHeader_2.54mm:PinHeader_1x03_P2.54mm_Vertical -> Potentiometer_THT:Potentiometer_Bourns_3339P_Vertical_HandSoldering
Changed lines of the file:
@@
 $Descr A4 11693 8268
 encoding utf-8
-Sheet 4 7
+Sheet 4 8
 Title ""
 Date ""
@@
 F 0 "C34" H 6365 5046 50  0000 L CNN
 F 1 ".0022" H 6365 4955 50  0000 L CNN
-F 2 "Capacitor_SMD:C_0805_2012Metric_Pad1.18x1.45mm_HandSolder" H 6288 4850 50  0001 C CNN
+F 2 "Capacitor_SMD:C_0805_2012Metric" H 6288 4850 50  0001 C CNN
 F 3 "~" H 6250 5000 50  0001 C CNN
 	1    6250 5000
@@
 F 0 "Q8" H 5591 5046 50  0000 L CNN
 F 1 "Q_NPN_BCE" H 5591 4955 50  0000 L CNN
-F 2 "Package_TO_SOT_SMD:SOT-23" H 5600 5100 50  0001 C CNN
+F 2 "Package_TO_SOT_SMD:SOT-89-3" H 5600 5100 50  0001 C CNN
 F 3 "~" H 5400 5000 50  0001 C CNN
 	1    5400 5000
@@
 F 0 "Q9" H 7091 5046 50  0000 L CNN
 F 1 "Q_NPN_BCE" H 7091 4955 50  0000 L CNN
-F 2 "Package_TO_SOT_SMD:SOT-23" H 7100 5100 50  0001 C CNN
+F 2 "Package_TO_SOT_SMD:SOT-89-3" H 7100 5100 50  0001 C CNN
 F 3 "~" H 6900 5000 50  0001 C CNN
 	1    6900 5000
@@
 F 0 "R51" H 6570 4796 50  0000 L CNN
 F 1 "2.2M" H 6570 4705 50  0000 L CNN
-F 2 "Resistor_SMD:R_0805_2012Metric_Pad1.20x1.40mm_HandSolder" V 6430 4750 50  0001 C CNN
+F 2 "Resistor_SMD:R_0805_2012Metric" V 6430 4750 50  0001 C CNN
 F 3 "~" H 6500 4750 50  0001 C CNN
 	1    6500 4750
@@
 F 0 "R50" H 5070 4796 50  0000 L CNN
 F 1 "2.2M" H 5070 4705 50  0000 L CNN
-F 2 "Resistor_SMD:R_0805_2012Metric_Pad1.20x1.40mm_HandSolder" V 4930 4750 50  0001 C CNN
+F 2 "Resistor_SMD:R_0805_2012Metric" V 4930 4750 50  0001 C CNN
 F 3 "~" H 5000 4750 50  0001 C CNN
 	1    5000 4750
@@
 F 0 "R49" H 6320 4046 50  0000 L CNN
 F 1 "10k" H 6320 3955 50  0000 L CNN
-F 2 "Resistor_SMD:R_0805_2012Metric_Pad1.20x1.40mm_HandSolder" V 6180 4000 50  0001 C CNN
+F 2 "Resistor_SMD:R_0805_2012Metric" V 6180 4000 50  0001 C CNN
 F 3 "~" H 6250 4000 50  0001 C CNN
 	1    6250 4000
@@
 F 0 "R24" H 8320 4046 50  0000 L CNN
 F 1 "1K" H 8320 3955 50  0000 L CNN
-F 2 "Resistor_SMD:R_0805_2012Metric_Pad1.20x1.40mm_HandSolder" V 8180 4000 50  0001 C CNN
+F 2 "Resistor_SMD:R_0805_2012Metric" V 8180 4000 50  0001 C CNN
 F 3 "~" H 8250 4000 50  0001 C CNN
 	1    8250 4000
@@
 F 0 "C14" H 8118 4796 50  0000 L CNN
 F 1 "22/10" H 8118 4705 50  0000 L CNN
-F 2 "Connector_PinHeader_2.54mm:PinHeader_1x02_P2.54mm_Vertical" H 8038 4600 50  0001 C CNN
+F 2 "Capacitor_THT:CP_Radial_D5.0mm_P2.50mm" H 8038 4600 50  0001 C CNN
 F 3 "~" H 8000 4750 50  0001 C CNN
 	1    8000 4750
@@
 F 0 "VR7" H 6930 4296 50  0000 R CNN
 F 1 "10kB" H 6930 4205 50  0000 R CNN
-F 2 "Connector_PinHeader_2.54mm:PinHeader_1x03_P2.54mm_Vertical" H 7000 4250 50  0001 C CNN
+F 2 "Potentiometer_THT:Potentiometer_Bourns_3339P_Vertical_HandSoldering" H 7000 4250 50  0001 C CNN
 F 3 "~" H 7000 4250 50  0001 C CNN
 	1    7000 4250
