File: DR-55-OUT/DR-55-OUT.sch (KiCad schematic (older format))
At the start: 21 parts

Commit message: Output finished
Finished the output schematic and routed alll the traces between the submodules
Parts:
- removed C?: C, symbol Device:C
- removed C?: CP, symbol Device:CP
- removed D?: D, symbol Device:D
- removed Q?: Q_NPN_BCE, symbol Device:Q_NPN_BCE
- removed R?: R, symbol Device:R
- added C?: C, symbol Device:C
- added C? (x4): CP, symbol Device:CP
- added Q?: Q_NPN_BCE, symbol Device:Q_NPN_BCE
- added R? (x6): R, symbol Device:R
- added R?: RTRIM, symbol Device:RTRIM
- added RV?: R_POT_TRIM, symbol Device:R_POT_TRIM
Connections:
- net labels added: Noisyout-IN
- wire segments 35 -> 75

Commit message: Values
Added Values to all components
Parts:
- C?: value CP -> .15/35
- C? (x4): value CP -> 4.7/35
- C? (x2): value CP -> 22/10
- C?: value C -> .0018
- R? (x3): value R -> 1k
- R?: value R -> 680k
- R?: value RTRIM -> 500kC
- R? (x2): value R -> 2.2M
- R?: value R -> 47k
- R? (x2): value R -> 100k
- R? (x2): value R -> 68k
- R?: value R -> 22k
- R?: value R -> 10k
- R?: value R -> 100
- R?: value RTRIM -> 1MA
- RV?: value R_POT_TRIM -> 10kA
Changed lines of the file:
@@
 $Descr A4 11693 8268
 encoding utf-8
-Sheet 6 7
+Sheet 5 7
 Title ""
 Date ""
@@
 AR Path="/627A1DA3/627AB13F" Ref="R?"  Part="1"
 F 0 "R?" H 2320 3046 50  0000 L CNN
-F 1 "R" H 2320 2955 50  0000 L CNN
+F 1 "1k" H 2320 2955 50  0000 L CNN
 F 2 "" V 2180 3000 50  0001 C CNN
 F 3 "~" H 2250 3000 50  0001 C CNN
@@
 AR Path="/627A1DA3/627B320F" Ref="C?"  Part="1"
 F 0 "C?" H 2618 3296 50  0000 L CNN
-F 1 "CP" H 2618 3205 50  0000 L CNN
+F 1 ".15/35" H 2618 3205 50  0000 L CNN
 F 2 "" H 2538 3100 50  0001 C CNN
 F 3 "~" H 2500 3250 50  0001 C CNN
@@
 AR Path="/627A1DA3/627B6EC6" Ref="R?"  Part="1"
 F 0 "R?" H 3070 3296 50  0000 L CNN
-F 1 "R" H 3070 3205 50  0000 L CNN
+F 1 "680k" H 3070 3205 50  0000 L CNN
 F 2 "" V 2930 3250 50  0001 C CNN
 F 3 "~" H 3000 3250 50  0001 C CNN
@@
 P 2500 1750
 F 0 "R?" H 2628 1796 50  0000 L CNN
-F 1 "RTRIM" H 2628 1705 50  0000 L CNN
+F 1 "500kC" H 2628 1705 50  0000 L CNN
 F 2 "" V 2430 1750 50  0001 C CNN
 F 3 "~" H 2500 1750 50  0001 C CNN
@@
 AR Path="/627A1DA3/627BF099" Ref="R?"  Part="1"
 F 0 "R?" H 3570 2546 50  0000 L CNN
-F 1 "R" H 3570 2455 50  0000 L CNN
+F 1 "2.2M" H 3570 2455 50  0000 L CNN
 F 2 "" V 3430 2500 50  0001 C CNN
 F 3 "~" H 3500 2500 50  0001 C CNN
@@
 AR Path="/627A1DA3/627C1BFC" Ref="C?"  Part="1"
 F 0 "C?" H 2368 1546 50  0000 L CNN
-F 1 "CP" H 2368 1455 50  0000 L CNN
+F 1 "4.7/35" H 2368 1455 50  0000 L CNN
 F 2 "" H 2288 1350 50  0001 C CNN
 F 3 "~" H 2250 1500 50  0001 C CNN
@@
 AR Path="/627A1DA3/627C2326" Ref="R?"  Part="1"
 F 0 "R?" H 2070 1796 50  0000 L CNN
-F 1 "R" H 2070 1705 50  0000 L CNN
+F 1 "47k" H 2070 1705 50  0000 L CNN
 F 2 "" V 1930 1750 50  0001 C CNN
 F 3 "~" H 2000 1750 50  0001 C CNN
@@
 AR Path="/627A1DA3/627C2CC6" Ref="R?"  Part="1"
 F 0 "R?" H 3070 1546 50  0000 L CNN
-F 1 "R" H 3070 1455 50  0000 L CNN
+F 1 "100k" H 3070 1455 50  0000 L CNN
 F 2 "" V 2930 1500 50  0001 C CNN
 F 3 "~" H 3000 1500 50  0001 C CNN
@@
 AR Path="/627A1DA3/627C2F5B" Ref="R?"  Part="1"
 F 0 "R?" H 3820 1546 50  0000 L CNN
-F 1 "R" H 3820 1455 50  0000 L CNN
+F 1 "68k" H 3820 1455 50  0000 L CNN
 F 2 "" V 3680 1500 50  0001 C CNN
 F 3 "~" H 3750 1500 50  0001 C CNN
@@
 AR Path="/627A1DA3/627C63AF" Ref="C?"  Part="1"
 F 0 "C?" H 4118 2796 50  0000 L CNN
-F 1 "CP" H 4118 2705 50  0000 L CNN
+F 1 "22/10" H 4118 2705 50  0000 L CNN
 F 2 "" H 4038 2600 50  0001 C CNN
 F 3 "~" H 4000 2750 50  0001 C CNN
@@
 AR Path="/627A1DA3/627C6E6F" Ref="R?"  Part="1"
 F 0 "R?" H 5070 1296 50  0000 L CNN
-F 1 "R" H 5070 1205 50  0000 L CNN
+F 1 "22k" H 5070 1205 50  0000 L CNN
 F 2 "" V 4930 1250 50  0001 C CNN
 F 3 "~" H 5000 1250 50  0001 C CNN
@@
 AR Path="/627A1DA3/627C72BD" Ref="R?"  Part="1"
 F 0 "R?" H 5070 1796 50  0000 L CNN
-F 1 "R" H 5070 1705 50  0000 L CNN
+F 1 "68k" H 5070 1705 50  0000 L CNN
 F 2 "" V 4930 1750 50  0001 C CNN
 F 3 "~" H 5000 1750 50  0001 C CNN
@@
 AR Path="/627A1DA3/6281E074" Ref="R?"  Part="1"
 F 0 "R?" H 5570 4796 50  0000 L CNN
-F 1 "R" H 5570 4705 50  0000 L CNN
+F 1 "10k" H 5570 4705 50  0000 L CNN
 F 2 "" V 5430 4750 50  0001 C CNN
 F 3 "~" H 5500 4750 50  0001 C CNN
@@
 AR Path="/627A1DA3/6281EC37" Ref="C?"  Part="1"
 F 0 "C?" H 5115 5046 50  0000 L CNN
-F 1 "C" H 5115 4955 50  0000 L CNN
+F 1 ".0018" H 5115 4955 50  0000 L CNN
 F 2 "" H 5038 4850 50  0001 C CNN
 F 3 "~" H 5000 5000 50  0001 C CNN
@@
 AR Path="/627A1DA3/6281F3FA" Ref="R?"  Part="1"
 F 0 "R?" H 5070 5796 50  0000 L CNN
-F 1 "R" H 5070 5705 50  0000 L CNN
+F 1 "2.2M" H 5070 5705 50  0000 L CNN
 F 2 "" V 4930 5750 50  0001 C CNN
 F 3 "~" H 5000 5750 50  0001 C CNN
@@
 AR Path="/627A1DA3/62821AD2" Ref="C?"  Part="1"
 F 0 "C?" H 5868 5546 50  0000 L CNN
-F 1 "CP" H 5868 5455 50  0000 L CNN
+F 1 "4.7/35" H 5868 5455 50  0000 L CNN
 F 2 "" H 5788 5350 50  0001 C CNN
 F 3 "~" H 5750 5500 50  0001 C CNN
@@
 AR Path="/627A1DA3/62824C07" Ref="R?"  Part="1"
 F 0 "R?" H 5570 6796 50  0000 L CNN
-F 1 "R" H 5570 6705 50  0000 L CNN
+F 1 "100" H 5570 6705 50  0000 L CNN
 F 2 "" V 5430 6750 50  0001 C CNN
 F 3 "~" H 5500 6750 50  0001 C CNN
@@
 AR Path="/627A1DA3/62825E6B" Ref="R?"  Part="1"
 F 0 "R?" H 6070 5796 50  0000 L CNN
-F 1 "R" H 6070 5705 50  0000 L CNN
+F 1 "100k" H 6070 5705 50  0000 L CNN
 F 2 "" V 5930 5750 50  0001 C CNN
 F 3 "~" H 6000 5750 50  0001 C CNN
@@
 AR Path="/627A1DA3/62827240" Ref="C?"  Part="1"
 F 0 "C?" H 6118 4796 50  0000 L CNN
-F 1 "CP" H 6118 4705 50  0000 L CNN
+F 1 "22/10" H 6118 4705 50  0000 L CNN
 F 2 "" H 6038 4600 50  0001 C CNN
 F 3 "~" H 6000 4750 50  0001 C CNN
@@
 AR Path="/627A1DA3/62827ACA" Ref="R?"  Part="1"
 F 0 "R?" H 6070 4296 50  0000 L CNN
-F 1 "R" H 6070 4205 50  0000 L CNN
+F 1 "1k" H 6070 4205 50  0000 L CNN
 F 2 "" V 5930 4250 50  0001 C CNN
 F 3 "~" H 6000 4250 50  0001 C CNN
@@
 P 4500 5500
 F 0 "R?" H 4628 5546 50  0000 L CNN
-F 1 "RTRIM" H 4628 5455 50  0000 L CNN
+F 1 "1MA" H 4628 5455 50  0000 L CNN
 F 2 "" V 4430 5500 50  0001 C CNN
 F 3 "~" H 4500 5500 50  0001 C CNN
@@
 AR Path="/627A1DA3/6283321B" Ref="C?"  Part="1"
 F 0 "C?" H 4368 6046 50  0000 L CNN
-F 1 "CP" H 4368 5955 50  0000 L CNN
+F 1 "4.7/35" H 4368 5955 50  0000 L CNN
 F 2 "" H 4288 5850 50  0001 C CNN
 F 3 "~" H 4250 6000 50  0001 C CNN
@@
 AR Path="/627A1DA3/62835074" Ref="R?"  Part="1"
 F 0 "R?" H 4070 5546 50  0000 L CNN
-F 1 "R" H 4070 5455 50  0000 L CNN
+F 1 "1k" H 4070 5455 50  0000 L CNN
 F 2 "" V 3930 5500 50  0001 C CNN
 F 3 "~" H 4000 5500 50  0001 C CNN
@@
 AR Path="/627A1DA3/6283956B" Ref="RV?"  Part="1"
 F 0 "RV?" H 3430 5046 50  0000 R CNN
-F 1 "R_POT_TRIM" H 3430 4955 50  0000 R CNN
+F 1 "10kA" H 3430 4955 50  0000 R CNN
 F 2 "" H 3500 5000 50  0001 C CNN
 F 3 "~" H 3500 5000 50  0001 C CNN
@@
 AR Path="/627A1DA3/6283A921" Ref="C?"  Part="1"
 F 0 "C?" H 4368 4546 50  0000 L CNN
-F 1 "CP" H 4368 4455 50  0000 L CNN
+F 1 "4.7/35" H 4368 4455 50  0000 L CNN
 F 2 "" H 4288 4350 50  0001 C CNN
 F 3 "~" H 4250 4500 50  0001 C CNN

Commit message: Resistor enumeration
All resistors, diodes and transistors get numbers
Parts:
- gave numbers to parts that had none: 21
Changed lines of the file:
@@
 $Descr A4 11693 8268
 encoding utf-8
-Sheet 5 7
+Sheet 7 7
 Title ""
 Date ""
@@
 AR Path="/62740CD0/627AB13F" Ref="R?"  Part="1"
 AR Path="/62804339/627AB13F" Ref="R?"  Part="1"
-AR Path="/627A1DA3/627AB13F" Ref="R?"  Part="1"
-F 0 "R?" H 2320 3046 50  0000 L CNN
+AR Path="/627A1DA3/627AB13F" Ref="R60"  Part="1"
+F 0 "R60" H 2320 3046 50  0000 L CNN
 F 1 "1k" H 2320 2955 50  0000 L CNN
 F 2 "" V 2180 3000 50  0001 C CNN
@@
 AR Path="/62740CD0/627AB1A8" Ref="D?"  Part="1"
 AR Path="/62804339/627AB1A8" Ref="D?"  Part="1"
-AR Path="/627A1DA3/627AB1A8" Ref="D?"  Part="1"
-F 0 "D?" V 1796 2920 50  0000 R CNN
+AR Path="/627A1DA3/627AB1A8" Ref="D1"  Part="1"
+F 0 "D1" V 1796 2920 50  0000 R CNN
 F 1 "D" V 1705 2920 50  0000 R CNN
 F 2 "" H 1750 3000 50  0001 C CNN
@@
 AR Path="/62740CD0/627B6EC6" Ref="R?"  Part="1"
 AR Path="/62804339/627B6EC6" Ref="R?"  Part="1"
-AR Path="/627A1DA3/627B6EC6" Ref="R?"  Part="1"
-F 0 "R?" H 3070 3296 50  0000 L CNN
+AR Path="/627A1DA3/627B6EC6" Ref="R16"  Part="1"
+F 0 "R16" H 3070 3296 50  0000 L CNN
 F 1 "680k" H 3070 3205 50  0000 L CNN
 F 2 "" V 2930 3250 50  0001 C CNN
@@
 AR Path="/62740CD0/627B7798" Ref="D?"  Part="1"
 AR Path="/62804339/627B7798" Ref="D?"  Part="1"
-AR Path="/627A1DA3/627B7798" Ref="D?"  Part="1"
-F 0 "D?" V 3046 2670 50  0000 R CNN
+AR Path="/627A1DA3/627B7798" Ref="D2"  Part="1"
+F 0 "D2" V 3046 2670 50  0000 R CNN
 F 1 "D" V 2955 2670 50  0000 R CNN
 F 2 "" H 3000 2750 50  0001 C CNN
@@
 $EndComp
 $Comp
-L Device:RTRIM R?
+L Device:RTRIM VR4
 U 1 1 627B95DC
 P 2500 1750
-F 0 "R?" H 2628 1796 50  0000 L CNN
+F 0 "VR4" H 2628 1796 50  0000 L CNN
 F 1 "500kC" H 2628 1705 50  0000 L CNN
 F 2 "" V 2430 1750 50  0001 C CNN
@@
 $EndComp
 $Comp
-L Device:Q_NJFET_SGD Q?
+L Device:Q_NJFET_SGD Q3
 U 1 1 627BBF5F
 P 3000 2100
-F 0 "Q?" V 3328 2100 50  0000 C CNN
+F 0 "Q3" V 3328 2100 50  0000 C CNN
 F 1 "Q_NJFET_SGD" V 3237 2100 50  0000 C CNN
 F 2 "" H 3200 2200 50  0001 C CNN
@@
 AR Path="/62740CD0/627BF099" Ref="R?"  Part="1"
 AR Path="/62804339/627BF099" Ref="R?"  Part="1"
-AR Path="/627A1DA3/627BF099" Ref="R?"  Part="1"
-F 0 "R?" H 3570 2546 50  0000 L CNN
+AR Path="/627A1DA3/627BF099" Ref="R13"  Part="1"
+F 0 "R13" H 3570 2546 50  0000 L CNN
 F 1 "2.2M" H 3570 2455 50  0000 L CNN
 F 2 "" V 3430 2500 50  0001 C CNN
@@
 AR Path="/62740CD0/627C2326" Ref="R?"  Part="1"
 AR Path="/62804339/627C2326" Ref="R?"  Part="1"
-AR Path="/627A1DA3/627C2326" Ref="R?"  Part="1"
-F 0 "R?" H 2070 1796 50  0000 L CNN
+AR Path="/627A1DA3/627C2326" Ref="R39"  Part="1"
+F 0 "R39" H 2070 1796 50  0000 L CNN
 F 1 "47k" H 2070 1705 50  0000 L CNN
 F 2 "" V 1930 1750 50  0001 C CNN
@@
 AR Path="/62740CD0/627C2CC6" Ref="R?"  Part="1"
 AR Path="/62804339/627C2CC6" Ref="R?"  Part="1"
-AR Path="/627A1DA3/627C2CC6" Ref="R?"  Part="1"
-F 0 "R?" H 3070 1546 50  0000 L CNN
+AR Path="/627A1DA3/627C2CC6" Ref="R14"  Part="1"
+F 0 "R14" H 3070 1546 50  0000 L CNN
 F 1 "100k" H 3070 1455 50  0000 L CNN
 F 2 "" V 2930 1500 50  0001 C CNN
@@
 AR Path="/62740CD0/627C2F5B" Ref="R?"  Part="1"
 AR Path="/62804339/627C2F5B" Ref="R?"  Part="1"
-AR Path="/627A1DA3/627C2F5B" Ref="R?"  Part="1"
-F 0 "R?" H 3820 1546 50  0000 L CNN
+AR Path="/627A1DA3/627C2F5B" Ref="R15"  Part="1"
+F 0 "R15" H 3820 1546 50  0000 L CNN
 F 1 "68k" H 3820 1455 50  0000 L CNN
 F 2 "" V 3680 1500 50  0001 C CNN
@@
 AR Path="/62740CD0/627C6E6F" Ref="R?"  Part="1"
 AR Path="/62804339/627C6E6F" Ref="R?"  Part="1"
-AR Path="/627A1DA3/627C6E6F" Ref="R?"  Part="1"
-F 0 "R?" H 5070 1296 50  0000 L CNN
+AR Path="/627A1DA3/627C6E6F" Ref="R101"  Part="1"
+F 0 "R101" H 5070 1296 50  0000 L CNN
 F 1 "22k" H 5070 1205 50  0000 L CNN
 F 2 "" V 4930 1250 50  0001 C CNN
@@
 AR Path="/62740CD0/627C72BD" Ref="R?"  Part="1"
 AR Path="/62804339/627C72BD" Ref="R?"  Part="1"
-AR Path="/627A1DA3/627C72BD" Ref="R?"  Part="1"
-F 0 "R?" H 5070 1796 50  0000 L CNN
+AR Path="/627A1DA3/627C72BD" Ref="R102"  Part="1"
+F 0 "R102" H 5070 1796 50  0000 L CNN
 F 1 "68k" H 5070 1705 50  0000 L CNN
 F 2 "" V 4930 1750 50  0001 C CNN
@@
 AR Path="/62740CD0/6281E074" Ref="R?"  Part="1"
 AR Path="/62804339/6281E074" Ref="R?"  Part="1"
-AR Path="/627A1DA3/6281E074" Ref="R?"  Part="1"
-F 0 "R?" H 5570 4796 50  0000 L CNN
+AR Path="/627A1DA3/6281E074" Ref="R19"  Part="1"
+F 0 "R19" H 5570 4796 50  0000 L CNN
 F 1 "10k" H 5570 4705 50  0000 L CNN
 F 2 "" V 5430 4750 50  0001 C CNN
@@
 AR Path="/62740CD0/6281F3FA" Ref="R?"  Part="1"
 AR Path="/62804339/6281F3FA" Ref="R?"  Part="1"
-AR Path="/627A1DA3/6281F3FA" Ref="R?"  Part="1"
-F 0 "R?" H 5070 5796 50  0000 L CNN
+AR Path="/627A1DA3/6281F3FA" Ref="R18"  Part="1"
+F 0 "R18" H 5070 5796 50  0000 L CNN
 F 1 "2.2M" H 5070 5705 50  0000 L CNN
 F 2 "" V 4930 5750 50  0001 C CNN
@@
 AR Path="/62740CD0/62822EB6" Ref="Q?"  Part="1"
 AR Path="/62804339/62822EB6" Ref="Q?"  Part="1"
-AR Path="/627A1DA3/62822EB6" Ref="Q?"  Part="1"
-F 0 "Q?" H 5591 6046 50  0000 L CNN
+AR Path="/627A1DA3/62822EB6" Ref="Q4"  Part="1"
+F 0 "Q4" H 5591 6046 50  0000 L CNN
 F 1 "Q_NPN_BCE" H 5591 5955 50  0000 L CNN
 F 2 "" H 5600 6100 50  0001 C CNN
@@
 AR Path="/62740CD0/62824C07" Ref="R?"  Part="1"
 AR Path="/62804339/62824C07" Ref="R?"  Part="1"
-AR Path="/627A1DA3/62824C07" Ref="R?"  Part="1"
-F 0 "R?" H 5570 6796 50  0000 L CNN
+AR Path="/627A1DA3/62824C07" Ref="R20"  Part="1"
+F 0 "R20" H 5570 6796 50  0000 L CNN
 F 1 "100" H 5570 6705 50  0000 L CNN
 F 2 "" V 5430 6750 50  0001 C CNN
@@
 AR Path="/62740CD0/62825E6B" Ref="R?"  Part="1"
 AR Path="/62804339/62825E6B" Ref="R?"  Part="1"
-AR Path="/627A1DA3/62825E6B" Ref="R?"  Part="1"
-F 0 "R?" H 6070 5796 50  0000 L CNN
+AR Path="/627A1DA3/62825E6B" Ref="R21"  Part="1"
+F 0 "R21" H 6070 5796 50  0000 L CNN
 F 1 "100k" H 6070 5705 50  0000 L CNN
 F 2 "" V 5930 5750 50  0001 C CNN
@@
 AR Path="/62740CD0/62827ACA" Ref="R?"  Part="1"
 AR Path="/62804339/62827ACA" Ref="R?"  Part="1"
-AR Path="/627A1DA3/62827ACA" Ref="R?"  Part="1"
-F 0 "R?" H 6070 4296 50  0000 L CNN
+AR Path="/627A1DA3/62827ACA" Ref="R22"  Part="1"
+F 0 "R22" H 6070 4296 50  0000 L CNN
 F 1 "1k" H 6070 4205 50  0000 L CNN
 F 2 "" V 5930 4250 50  0001 C CNN
@@
 	5000 6000 5000 5900
 $Comp
-L Device:RTRIM R?
+L Device:RTRIM VR1
 U 1 1 6282DE59
 P 4500 5500
-F 0 "R?" H 4628 5546 50  0000 L CNN
+F 0 "VR1" H 4628 5546 50  0000 L CNN
 F 1 "1MA" H 4628 5455 50  0000 L CNN
 F 2 "" V 4430 5500 50  0001 C CNN
@@
 AR Path="/62740CD0/62835074" Ref="R?"  Part="1"
 AR Path="/62804339/62835074" Ref="R?"  Part="1"
-AR Path="/627A1DA3/62835074" Ref="R?"  Part="1"
-F 0 "R?" H 4070 5546 50  0000 L CNN
+AR Path="/627A1DA3/62835074" Ref="R17"  Part="1"
+F 0 "R17" H 4070 5546 50  0000 L CNN
 F 1 "1k" H 4070 5455 50  0000 L CNN
 F 2 "" V 3930 5500 50  0001 C CNN
@@
 P 3500 5000
 AR Path="/62804B1F/6283956B" Ref="RV?"  Part="1"
-AR Path="/627A1DA3/6283956B" Ref="RV?"  Part="1"
-F 0 "RV?" H 3430 5046 50  0000 R CNN
+AR Path="/627A1DA3/6283956B" Ref="VR2"  Part="1"
+F 0 "VR2" H 3430 5046 50  0000 R CNN
 F 1 "10kA" H 3430 4955 50  0000 R CNN
 F 2 "" H 3500 5000 50  0001 C CNN

Commit message: Footprints added
Added most of the footprints for a 0805 SMD PCB. some placeholder footprints added and some missing
Parts:
- C10: renamed from C?; footprint (none) -> Capacitor_SMD:C_0805_2012Metric_Pad1.18x1.45mm_HandSolder
- D1: footprint (none) -> Diode_SMD:D_SOD-123F
- D2: footprint (none) -> Diode_SMD:D_SOD-123
- J7: renamed from J?; footprint (none) -> Connector_PinHeader_2.54mm:PinHeader_1x03_P2.54mm_Vertical
- Q3: footprint (none) -> Connector_PinHeader_2.54mm:PinHeader_1x03_P2.54mm_Vertical
- Q4: footprint (none) -> Package_TO_SOT_SMD:SOT-23
- R101, R102, R13, R14, R15, R16, R17, R18, R19, R20, R21, R22, R39, R60: footprint (none) -> Resistor_SMD:R_0805_2012Metric_Pad1.20x1.40mm_HandSolder
- gave numbers to parts that had none: 7

Commit message: SMD PCB
added all all Pcb layouts without CP footprint
Parts:
- C11, C12, C24, C6, C7, C8, C9: footprint (none) -> Connector_PinHeader_2.54mm:PinHeader_1x02_P2.54mm_Vertical
- J7: value Thonkiconn -> Accent OUT
- VR1, VR2, VR4: footprint (none) -> Connector_PinHeader_2.54mm:PinHeader_1x03_P2.54mm_Vertical
Changed lines of the file:
@@
 F 0 "C6" H 2618 3296 50  0000 L CNN
 F 1 ".15/35" H 2618 3205 50  0000 L CNN
-F 2 "" H 2538 3100 50  0001 C CNN
+F 2 "Connector_PinHeader_2.54mm:PinHeader_1x02_P2.54mm_Vertical" H 2538 3100 50  0001 C CNN
 F 3 "~" H 2500 3250 50  0001 C CNN
 	1    2500 3250
@@
 F 0 "VR4" H 2628 1796 50  0000 L CNN
 F 1 "500kC" H 2628 1705 50  0000 L CNN
-F 2 "" V 2430 1750 50  0001 C CNN
+F 2 "Connector_PinHeader_2.54mm:PinHeader_1x03_P2.54mm_Vertical" V 2430 1750 50  0001 C CNN
 F 3 "~" H 2500 1750 50  0001 C CNN
 	1    2500 1750
@@
 F 0 "C24" H 2368 1546 50  0000 L CNN
 F 1 "4.7/35" H 2368 1455 50  0000 L CNN
-F 2 "" H 2288 1350 50  0001 C CNN
+F 2 "Connector_PinHeader_2.54mm:PinHeader_1x02_P2.54mm_Vertical" H 2288 1350 50  0001 C CNN
 F 3 "~" H 2250 1500 50  0001 C CNN
 	1    2250 1500
@@
 F 0 "C7" H 4118 2796 50  0000 L CNN
 F 1 "22/10" H 4118 2705 50  0000 L CNN
-F 2 "" H 4038 2600 50  0001 C CNN
+F 2 "Connector_PinHeader_2.54mm:PinHeader_1x02_P2.54mm_Vertical" H 4038 2600 50  0001 C CNN
 F 3 "~" H 4000 2750 50  0001 C CNN
 	1    4000 2750
@@
 P 3500 3000
 F 0 "J7" H 3350 3050 50  0000 L CNN
-F 1 "Thonkiconn" H 3350 3150 50  0000 L CNN
+F 1 "Accent OUT" H 3350 3150 50  0000 L CNN
 F 2 "Connector_PinHeader_2.54mm:PinHeader_1x03_P2.54mm_Vertical" H 3300 3200 50  0001 C CNN
 F 3 "" H 3300 3200 50  0001 C CNN
@@
 F 0 "C11" H 5868 5546 50  0000 L CNN
 F 1 "4.7/35" H 5868 5455 50  0000 L CNN
-F 2 "" H 5788 5350 50  0001 C CNN
+F 2 "Connector_PinHeader_2.54mm:PinHeader_1x02_P2.54mm_Vertical" H 5788 5350 50  0001 C CNN
 F 3 "~" H 5750 5500 50  0001 C CNN
 	1    5750 5500
@@
 F 0 "C12" H 6118 4796 50  0000 L CNN
 F 1 "22/10" H 6118 4705 50  0000 L CNN
-F 2 "" H 6038 4600 50  0001 C CNN
+F 2 "Connector_PinHeader_2.54mm:PinHeader_1x02_P2.54mm_Vertical" H 6038 4600 50  0001 C CNN
 F 3 "~" H 6000 4750 50  0001 C CNN
 	1    6000 4750
@@
 F 0 "VR1" H 4628 5546 50  0000 L CNN
 F 1 "1MA" H 4628 5455 50  0000 L CNN
-F 2 "" V 4430 5500 50  0001 C CNN
+F 2 "Connector_PinHeader_2.54mm:PinHeader_1x03_P2.54mm_Vertical" V 4430 5500 50  0001 C CNN
 F 3 "~" H 4500 5500 50  0001 C CNN
 	1    4500 5500
@@
 F 0 "C9" H 4368 6046 50  0000 L CNN
 F 1 "4.7/35" H 4368 5955 50  0000 L CNN
-F 2 "" H 4288 5850 50  0001 C CNN
+F 2 "Connector_PinHeader_2.54mm:PinHeader_1x02_P2.54mm_Vertical" H 4288 5850 50  0001 C CNN
 F 3 "~" H 4250 6000 50  0001 C CNN
 	1    4250 6000
@@
 F 0 "VR2" H 3430 5046 50  0000 R CNN
 F 1 "10kA" H 3430 4955 50  0000 R CNN
-F 2 "" H 3500 5000 50  0001 C CNN
+F 2 "Connector_PinHeader_2.54mm:PinHeader_1x03_P2.54mm_Vertical" H 3500 5000 50  0001 C CNN
 F 3 "~" H 3500 5000 50  0001 C CNN
 	1    3500 5000
@@
 F 0 "C8" H 4368 4546 50  0000 L CNN
 F 1 "4.7/35" H 4368 4455 50  0000 L CNN
-F 2 "" H 4288 4350 50  0001 C CNN
+F 2 "Connector_PinHeader_2.54mm:PinHeader_1x02_P2.54mm_Vertical" H 4288 4350 50  0001 C CNN
 F 3 "~" H 4250 4500 50  0001 C CNN
 	1    4250 4500
