File: DR-55-OUT/DR-55-OUT.sch (KiCad schematic (older format))
At the start: 30 parts, among them J7 Accent OUT, Q3 Q_NJFET_SGD, Q4 Q_NPN_BCE

Commit message: changed some stuff
Parts:
- C10: footprint Capacitor_SMD:C_0805_2012Metric_Pad1.18x1.45mm_HandSolder -> Capacitor_SMD:C_0805_2012Metric
- C11, C12, C24, C6, C7, C8, C9: footprint Connector_PinHeader_2.54mm:PinHeader_1x02_P2.54mm_Vertical -> Capacitor_THT:CP_Radial_D5.0mm_P2.50mm
- D2: footprint Diode_SMD:D_SOD-123 -> Diode_SMD:D_SOD-123F
- J7: footprint Connector_PinHeader_2.54mm:PinHeader_1x03_P2.54mm_Vertical -> Connector_PinHeader_2.54mm:PinHeader_1x02_P2.54mm_Vertical; symbol Eurorack:Thonkiconn -> DR-55-rescue:Thonkiconn-Eurorack
- Q3: footprint Connector_PinHeader_2.54mm:PinHeader_1x03_P2.54mm_Vertical -> Package_TO_SOT_THT:TO-92L_HandSolder
- Q4: footprint Package_TO_SOT_SMD:SOT-23 -> Package_TO_SOT_SMD:SOT-89-3
- R101, R102, R13, R14, R15, R16, R17, R18, R19, R20, R21, R22, R39, R60: footprint Resistor_SMD:R_0805_2012Metric_Pad1.20x1.40mm_HandSolder -> Resistor_SMD:R_0805_2012Metric
- VR1, VR2, VR4: footprint Connector_PinHeader_2.54mm:PinHeader_1x03_P2.54mm_Vertical -> Potentiometer_THT:Potentiometer_Alpha_RD901F-40-00D_Single_Vertical
Changed lines of the file:
@@
 $Descr A4 11693 8268
 encoding utf-8
-Sheet 7 7
+Sheet 7 8
 Title ""
 Date ""
@@
 F 0 "R60" H 2320 3046 50  0000 L CNN
 F 1 "1k" H 2320 2955 50  0000 L CNN
-F 2 "Resistor_SMD:R_0805_2012Metric_Pad1.20x1.40mm_HandSolder" V 2180 3000 50  0001 C CNN
+F 2 "Resistor_SMD:R_0805_2012Metric" V 2180 3000 50  0001 C CNN
 F 3 "~" H 2250 3000 50  0001 C CNN
 	1    2250 3000
@@
 F 0 "C6" H 2618 3296 50  0000 L CNN
 F 1 ".15/35" H 2618 3205 50  0000 L CNN
-F 2 "Connector_PinHeader_2.54mm:PinHeader_1x02_P2.54mm_Vertical" H 2538 3100 50  0001 C CNN
+F 2 "Capacitor_THT:CP_Radial_D5.0mm_P2.50mm" H 2538 3100 50  0001 C CNN
 F 3 "~" H 2500 3250 50  0001 C CNN
 	1    2500 3250
@@
 F 0 "R16" H 3070 3296 50  0000 L CNN
 F 1 "680k" H 3070 3205 50  0000 L CNN
-F 2 "Resistor_SMD:R_0805_2012Metric_Pad1.20x1.40mm_HandSolder" V 2930 3250 50  0001 C CNN
+F 2 "Resistor_SMD:R_0805_2012Metric" V 2930 3250 50  0001 C CNN
 F 3 "~" H 3000 3250 50  0001 C CNN
 	1    3000 3250
@@
 F 0 "D2" V 3046 2670 50  0000 R CNN
 F 1 "D" V 2955 2670 50  0000 R CNN
-F 2 "Diode_SMD:D_SOD-123" H 3000 2750 50  0001 C CNN
+F 2 "Diode_SMD:D_SOD-123F" H 3000 2750 50  0001 C CNN
 F 3 "~" H 3000 2750 50  0001 C CNN
 	1    3000 2750
@@
 F 0 "VR4" H 2628 1796 50  0000 L CNN
 F 1 "500kC" H 2628 1705 50  0000 L CNN
-F 2 "Connector_PinHeader_2.54mm:PinHeader_1x03_P2.54mm_Vertical" V 2430 1750 50  0001 C CNN
+F 2 "Potentiometer_THT:Potentiometer_Alpha_RD901F-40-00D_Single_Vertical" V 2430 1750 50  0001 C CNN
 F 3 "~" H 2500 1750 50  0001 C CNN
 	1    2500 1750
@@
 F 0 "Q3" V 3328 2100 50  0000 C CNN
 F 1 "Q_NJFET_SGD" V 3237 2100 50  0000 C CNN
-F 2 "Connector_PinHeader_2.54mm:PinHeader_1x03_P2.54mm_Vertical" H 3200 2200 50  0001 C CNN
+F 2 "Package_TO_SOT_THT:TO-92L_HandSolder" H 3200 2200 50  0001 C CNN
 F 3 "~" H 3000 2100 50  0001 C CNN
 	1    3000 2100
@@
 F 0 "R13" H 3570 2546 50  0000 L CNN
 F 1 "2.2M" H 3570 2455 50  0000 L CNN
-F 2 "Resistor_SMD:R_0805_2012Metric_Pad1.20x1.40mm_HandSolder" V 3430 2500 50  0001 C CNN
+F 2 "Resistor_SMD:R_0805_2012Metric" V 3430 2500 50  0001 C CNN
 F 3 "~" H 3500 2500 50  0001 C CNN
 	1    3500 2500
@@
 F 0 "C24" H 2368 1546 50  0000 L CNN
 F 1 "4.7/35" H 2368 1455 50  0000 L CNN
-F 2 "Connector_PinHeader_2.54mm:PinHeader_1x02_P2.54mm_Vertical" H 2288 1350 50  0001 C CNN
+F 2 "Capacitor_THT:CP_Radial_D5.0mm_P2.50mm" H 2288 1350 50  0001 C CNN
 F 3 "~" H 2250 1500 50  0001 C CNN
 	1    2250 1500
@@
 F 0 "R39" H 2070 1796 50  0000 L CNN
 F 1 "47k" H 2070 1705 50  0000 L CNN
-F 2 "Resistor_SMD:R_0805_2012Metric_Pad1.20x1.40mm_HandSolder" V 1930 1750 50  0001 C CNN
+F 2 "Resistor_SMD:R_0805_2012Metric" V 1930 1750 50  0001 C CNN
 F 3 "~" H 2000 1750 50  0001 C CNN
 	1    2000 1750
@@
 F 0 "R14" H 3070 1546 50  0000 L CNN
 F 1 "100k" H 3070 1455 50  0000 L CNN
-F 2 "Resistor_SMD:R_0805_2012Metric_Pad1.20x1.40mm_HandSolder" V 2930 1500 50  0001 C CNN
+F 2 "Resistor_SMD:R_0805_2012Metric" V 2930 1500 50  0001 C CNN
 F 3 "~" H 3000 1500 50  0001 C CNN
 	1    3000 1500
@@
 F 0 "R15" H 3820 1546 50  0000 L CNN
 F 1 "68k" H 3820 1455 50  0000 L CNN
-F 2 "Resistor_SMD:R_0805_2012Metric_Pad1.20x1.40mm_HandSolder" V 3680 1500 50  0001 C CNN
+F 2 "Resistor_SMD:R_0805_2012Metric" V 3680 1500 50  0001 C CNN
 F 3 "~" H 3750 1500 50  0001 C CNN
 	1    3750 1500
@@
 F 0 "C7" H 4118 2796 50  0000 L CNN
 F 1 "22/10" H 4118 2705 50  0000 L CNN
-F 2 "Connector_PinHeader_2.54mm:PinHeader_1x02_P2.54mm_Vertical" H 4038 2600 50  0001 C CNN
+F 2 "Capacitor_THT:CP_Radial_D5.0mm_P2.50mm" H 4038 2600 50  0001 C CNN
 F 3 "~" H 4000 2750 50  0001 C CNN
 	1    4000 2750
@@
 F 0 "R101" H 5070 1296 50  0000 L CNN
 F 1 "22k" H 5070 1205 50  0000 L CNN
-F 2 "Resistor_SMD:R_0805_2012Metric_Pad1.20x1.40mm_HandSolder" V 4930 1250 50  0001 C CNN
+F 2 "Resistor_SMD:R_0805_2012Metric" V 4930 1250 50  0001 C CNN
 F 3 "~" H 5000 1250 50  0001 C CNN
 	1    5000 1250
@@
 F 0 "R102" H 5070 1796 50  0000 L CNN
 F 1 "68k" H 5070 1705 50  0000 L CNN
-F 2 "Resistor_SMD:R_0805_2012Metric_Pad1.20x1.40mm_HandSolder" V 4930 1750 50  0001 C CNN
+F 2 "Resistor_SMD:R_0805_2012Metric" V 4930 1750 50  0001 C CNN
 F 3 "~" H 5000 1750 50  0001 C CNN
 	1    5000 1750
@@
 	1500 3000 1600 3000
 $Comp
-L Eurorack:Thonkiconn J7
+L DR-55-rescue:Thonkiconn-Eurorack J7
 U 1 1 627D0284
 P 3500 3000
 F 0 "J7" H 3350 3050 50  0000 L CNN
 F 1 "Accent OUT" H 3350 3150 50  0000 L CNN
-F 2 "Connector_PinHeader_2.54mm:PinHeader_1x03_P2.54mm_Vertical" H 3300 3200 50  0001 C CNN
+F 2 "Connector_PinHeader_2.54mm:PinHeader_1x02_P2.54mm_Vertical" H 3300 3200 50  0001 C CNN
 F 3 "" H 3300 3200 50  0001 C CNN
 	1    3500 3000
@@
 F 0 "R19" H 5570 4796 50  0000 L CNN
 F 1 "10k" H 5570 4705 50  0000 L CNN
-F 2 "Resistor_SMD:R_0805_2012Metric_Pad1.20x1.40mm_HandSolder" V 5430 4750 50  0001 C CNN
+F 2 "Resistor_SMD:R_0805_2012Metric" V 5430 4750 50  0001 C CNN
 F 3 "~" H 5500 4750 50  0001 C CNN
 	1    5500 4750
@@
 F 0 "C10" H 5115 5046 50  0000 L CNN
 F 1 ".0018" H 5115 4955 50  0000 L CNN
-F 2 "Capacitor_SMD:C_0805_2012Metric_Pad1.18x1.45mm_HandSolder" H 5038 4850 50  0001 C CNN
+F 2 "Capacitor_SMD:C_0805_2012Metric" H 5038 4850 50  0001 C CNN
 F 3 "~" H 5000 5000 50  0001 C CNN
 	1    5000 5000
@@
 F 0 "R18" H 5070 5796 50  0000 L CNN
 F 1 "2.2M" H 5070 5705 50  0000 L CNN
-F 2 "Resistor_SMD:R_0805_2012Metric_Pad1.20x1.40mm_HandSolder" V 4930 5750 50  0001 C CNN
+F 2 "Resistor_SMD:R_0805_2012Metric" V 4930 5750 50  0001 C CNN
 F 3 "~" H 5000 5750 50  0001 C CNN
 	1    5000 5750
@@
 F 0 "C11" H 5868 5546 50  0000 L CNN
 F 1 "4.7/35" H 5868 5455 50  0000 L CNN
-F 2 "Connector_PinHeader_2.54mm:PinHeader_1x02_P2.54mm_Vertical" H 5788 5350 50  0001 C CNN
+F 2 "Capacitor_THT:CP_Radial_D5.0mm_P2.50mm" H 5788 5350 50  0001 C CNN
 F 3 "~" H 5750 5500 50  0001 C CNN
 	1    5750 5500
@@
 F 0 "Q4" H 5591 6046 50  0000 L CNN
 F 1 "Q_NPN_BCE" H 5591 5955 50  0000 L CNN
-F 2 "Package_TO_SOT_SMD:SOT-23" H 5600 6100 50  0001 C CNN
+F 2 "Package_TO_SOT_SMD:SOT-89-3" H 5600 6100 50  0001 C CNN
 F 3 "~" H 5400 6000 50  0001 C CNN
 	1    5400 6000
@@
 F 0 "R20" H 5570 6796 50  0000 L CNN
 F 1 "100" H 5570 6705 50  0000 L CNN
-F 2 "Resistor_SMD:R_0805_2012Metric_Pad1.20x1.40mm_HandSolder" V 5430 6750 50  0001 C CNN
+F 2 "Resistor_SMD:R_0805_2012Metric" V 5430 6750 50  0001 C CNN
 F 3 "~" H 5500 6750 50  0001 C CNN
 	1    5500 6750
@@
 F 0 "R21" H 6070 5796 50  0000 L CNN
 F 1 "100k" H 6070 5705 50  0000 L CNN
-F 2 "Resistor_SMD:R_0805_2012Metric_Pad1.20x1.40mm_HandSolder" V 5930 5750 50  0001 C CNN
+F 2 "Resistor_SMD:R_0805_2012Metric" V 5930 5750 50  0001 C CNN
 F 3 "~" H 6000 5750 50  0001 C CNN
 	1    6000 5750
@@
 F 0 "C12" H 6118 4796 50  0000 L CNN
 F 1 "22/10" H 6118 4705 50  0000 L CNN
-F 2 "Connector_PinHeader_2.54mm:PinHeader_1x02_P2.54mm_Vertical" H 6038 4600 50  0001 C CNN
+F 2 "Capacitor_THT:CP_Radial_D5.0mm_P2.50mm" H 6038 4600 50  0001 C CNN
 F 3 "~" H 6000 4750 50  0001 C CNN
 	1    6000 4750
@@
 F 0 "R22" H 6070 4296 50  0000 L CNN
 F 1 "1k" H 6070 4205 50  0000 L CNN
-F 2 "Resistor_SMD:R_0805_2012Metric_Pad1.20x1.40mm_HandSolder" V 5930 4250 50  0001 C CNN
+F 2 "Resistor_SMD:R_0805_2012Metric" V 5930 4250 50  0001 C CNN
 F 3 "~" H 6000 4250 50  0001 C CNN
 	1    6000 4250
@@
 F 0 "VR1" H 4628 5546 50  0000 L CNN
 F 1 "1MA" H 4628 5455 50  0000 L CNN
-F 2 "Connector_PinHeader_2.54mm:PinHeader_1x03_P2.54mm_Vertical" V 4430 5500 50  0001 C CNN
+F 2 "Potentiometer_THT:Potentiometer_Alpha_RD901F-40-00D_Single_Vertical" V 4430 5500 50  0001 C CNN
 F 3 "~" H 4500 5500 50  0001 C CNN
 	1    4500 5500
@@
 F 0 "C9" H 4368 6046 50  0000 L CNN
 F 1 "4.7/35" H 4368 5955 50  0000 L CNN
-F 2 "Connector_PinHeader_2.54mm:PinHeader_1x02_P2.54mm_Vertical" H 4288 5850 50  0001 C CNN
+F 2 "Capacitor_THT:CP_Radial_D5.0mm_P2.50mm" H 4288 5850 50  0001 C CNN
 F 3 "~" H 4250 6000 50  0001 C CNN
 	1    4250 6000
@@
 F 0 "R17" H 4070 5546 50  0000 L CNN
 F 1 "1k" H 4070 5455 50  0000 L CNN
-F 2 "Resistor_SMD:R_0805_2012Metric_Pad1.20x1.40mm_HandSolder" V 3930 5500 50  0001 C CNN
+F 2 "Resistor_SMD:R_0805_2012Metric" V 3930 5500 50  0001 C CNN
 F 3 "~" H 4000 5500 50  0001 C CNN
 	1    4000 5500
@@
 F 0 "VR2" H 3430 5046 50  0000 R CNN
 F 1 "10kA" H 3430 4955 50  0000 R CNN
-F 2 "Connector_PinHeader_2.54mm:PinHeader_1x03_P2.54mm_Vertical" H 3500 5000 50  0001 C CNN
+F 2 "Potentiometer_THT:Potentiometer_Alpha_RD901F-40-00D_Single_Vertical" H 3500 5000 50  0001 C CNN
 F 3 "~" H 3500 5000 50  0001 C CNN
 	1    3500 5000
@@
 F 0 "C8" H 4368 4546 50  0000 L CNN
 F 1 "4.7/35" H 4368 4455 50  0000 L CNN
-F 2 "Connector_PinHeader_2.54mm:PinHeader_1x02_P2.54mm_Vertical" H 4288 4350 50  0001 C CNN
+F 2 "Capacitor_THT:CP_Radial_D5.0mm_P2.50mm" H 4288 4350 50  0001 C CNN
 F 3 "~" H 4250 4500 50  0001 C CNN
 	1    4250 4500
