File: DR-55-Rim/DR-55-Rim.sch (KiCad schematic (older format))
At the start: 17 parts

Commit message: Values
Added Values to all components
Parts:
- C? (x2): value C -> .0022
- C? (x2): value C -> .0015
- C?: value C -> 47p
- C?: value C -> .0027
- R?: value R -> 47k
- R?: value R -> 10k
- R?: value R -> 2.2M
- R?: value R -> 270
- R? (x2): value R -> 22k
- R?: value R -> 100k
- R? (x2): value R -> 33k
Changed lines of the file:
@@
 $Descr A4 11693 8268
 encoding utf-8
-Sheet 4 7
+Sheet 3 7
 Title ""
 Date ""
@@
 AR Path="/62804339/6280F25A" Ref="R?"  Part="1"
 F 0 "R?" H 4820 3546 50  0000 L CNN
-F 1 "R" H 4820 3455 50  0000 L CNN
+F 1 "47k" H 4820 3455 50  0000 L CNN
 F 2 "" V 4680 3500 50  0001 C CNN
 F 3 "~" H 4750 3500 50  0001 C CNN
@@
 AR Path="/62804339/62824005" Ref="R?"  Part="1"
 F 0 "R?" H 4570 3296 50  0000 L CNN
-F 1 "R" H 4570 3205 50  0000 L CNN
+F 1 "10k" H 4570 3205 50  0000 L CNN
 F 2 "" V 4430 3250 50  0001 C CNN
 F 3 "~" H 4500 3250 50  0001 C CNN
@@
 AR Path="/62804339/628244CD" Ref="R?"  Part="1"
 F 0 "R?" H 4070 3796 50  0000 L CNN
-F 1 "R" H 4070 3705 50  0000 L CNN
+F 1 "2.2M" H 4070 3705 50  0000 L CNN
 F 2 "" V 3930 3750 50  0001 C CNN
 F 3 "~" H 4000 3750 50  0001 C CNN
@@
 AR Path="/62804339/62825704" Ref="R?"  Part="1"
 F 0 "R?" H 4570 4796 50  0000 L CNN
-F 1 "R" H 4570 4705 50  0000 L CNN
+F 1 "270" H 4570 4705 50  0000 L CNN
 F 2 "" V 4430 4750 50  0001 C CNN
 F 3 "~" H 4500 4750 50  0001 C CNN
@@
 AR Path="/62804339/6282665D" Ref="R?"  Part="1"
 F 0 "R?" H 3570 4296 50  0000 L CNN
-F 1 "R" H 3570 4205 50  0000 L CNN
+F 1 "22k" H 3570 4205 50  0000 L CNN
 F 2 "" V 3430 4250 50  0001 C CNN
 F 3 "~" H 3500 4250 50  0001 C CNN
@@
 AR Path="/62804339/628267EC" Ref="R?"  Part="1"
 F 0 "R?" H 3070 4296 50  0000 L CNN
-F 1 "R" H 3070 4205 50  0000 L CNN
+F 1 "22k" H 3070 4205 50  0000 L CNN
 F 2 "" V 2930 4250 50  0001 C CNN
 F 3 "~" H 3000 4250 50  0001 C CNN
@@
 AR Path="/62804339/62826CDD" Ref="R?"  Part="1"
 F 0 "R?" H 2070 4296 50  0000 L CNN
-F 1 "R" H 2070 4205 50  0000 L CNN
+F 1 "100k" H 2070 4205 50  0000 L CNN
 F 2 "" V 1930 4250 50  0001 C CNN
 F 3 "~" H 2000 4250 50  0001 C CNN
@@
 AR Path="/62804339/62826FC4" Ref="R?"  Part="1"
 F 0 "R?" H 1570 4296 50  0000 L CNN
-F 1 "R" H 1570 4205 50  0000 L CNN
+F 1 "33k" H 1570 4205 50  0000 L CNN
 F 2 "" V 1430 4250 50  0001 C CNN
 F 3 "~" H 1500 4250 50  0001 C CNN
@@
 AR Path="/62804339/628275F6" Ref="C?"  Part="1"
 F 0 "C?" H 5365 3546 50  0000 L CNN
-F 1 "C" H 5365 3455 50  0000 L CNN
+F 1 ".0022" H 5365 3455 50  0000 L CNN
 F 2 "" H 5288 3350 50  0001 C CNN
 F 3 "~" H 5250 3500 50  0001 C CNN
@@
 AR Path="/62804339/62827C65" Ref="C?"  Part="1"
 F 0 "C?" H 3615 3546 50  0000 L CNN
-F 1 "C" H 3615 3455 50  0000 L CNN
+F 1 ".0022" H 3615 3455 50  0000 L CNN
 F 2 "" H 3538 3350 50  0001 C CNN
 F 3 "~" H 3500 3500 50  0001 C CNN
@@
 AR Path="/62804339/628283B5" Ref="C?"  Part="1"
 F 0 "C?" H 3365 4046 50  0000 L CNN
-F 1 "C" H 3365 3955 50  0000 L CNN
+F 1 ".0015" H 3365 3955 50  0000 L CNN
 F 2 "" H 3288 3850 50  0001 C CNN
 F 3 "~" H 3250 4000 50  0001 C CNN
@@
 AR Path="/62804339/62828526" Ref="C?"  Part="1"
 F 0 "C?" H 3865 4046 50  0000 L CNN
-F 1 "C" H 3865 3955 50  0000 L CNN
+F 1 ".0015" H 3865 3955 50  0000 L CNN
 F 2 "" H 3788 3850 50  0001 C CNN
 F 3 "~" H 3750 4000 50  0001 C CNN
@@
 AR Path="/62804339/62828F17" Ref="C?"  Part="1"
 F 0 "C?" H 2615 4296 50  0000 L CNN
-F 1 "C" H 2615 4205 50  0000 L CNN
+F 1 "47p" H 2615 4205 50  0000 L CNN
 F 2 "" H 2538 4100 50  0001 C CNN
 F 3 "~" H 2500 4250 50  0001 C CNN
@@
 AR Path="/62804339/62829280" Ref="C?"  Part="1"
 F 0 "C?" H 1865 4046 50  0000 L CNN
-F 1 "C" H 1865 3955 50  0000 L CNN
+F 1 ".0027" H 1865 3955 50  0000 L CNN
 F 2 "" H 1788 3850 50  0001 C CNN
 F 3 "~" H 1750 4000 50  0001 C CNN
@@
 AR Path="/62804339/62829D12" Ref="R?"  Part="1"
 F 0 "R?" H 2320 4046 50  0000 L CNN
-F 1 "R" H 2320 3955 50  0000 L CNN
+F 1 "33k" H 2320 3955 50  0000 L CNN
 F 2 "" V 2180 4000 50  0001 C CNN
 F 3 "~" H 2250 4000 50  0001 C CNN

Commit message: Resistor enumeration
All resistors, diodes and transistors get numbers
Parts:
- gave numbers to parts that had none: 11
Changed lines of the file:
@@
 P 4750 3500
 AR Path="/62740CD0/6280F25A" Ref="R?"  Part="1"
-AR Path="/62804339/6280F25A" Ref="R?"  Part="1"
-F 0 "R?" H 4820 3546 50  0000 L CNN
+AR Path="/62804339/6280F25A" Ref="R41"  Part="1"
+F 0 "R41" H 4820 3546 50  0000 L CNN
 F 1 "47k" H 4820 3455 50  0000 L CNN
 F 2 "" V 4680 3500 50  0001 C CNN
@@
 P 4500 3250
 AR Path="/62740CD0/62824005" Ref="R?"  Part="1"
-AR Path="/62804339/62824005" Ref="R?"  Part="1"
-F 0 "R?" H 4570 3296 50  0000 L CNN
+AR Path="/62804339/62824005" Ref="R40"  Part="1"
+F 0 "R40" H 4570 3296 50  0000 L CNN
 F 1 "10k" H 4570 3205 50  0000 L CNN
 F 2 "" V 4430 3250 50  0001 C CNN
@@
 P 4000 3750
 AR Path="/62740CD0/628244CD" Ref="R?"  Part="1"
-AR Path="/62804339/628244CD" Ref="R?"  Part="1"
-F 0 "R?" H 4070 3796 50  0000 L CNN
+AR Path="/62804339/628244CD" Ref="R43"  Part="1"
+F 0 "R43" H 4070 3796 50  0000 L CNN
 F 1 "2.2M" H 4070 3705 50  0000 L CNN
 F 2 "" V 3930 3750 50  0001 C CNN
@@
 P 4500 4750
 AR Path="/62740CD0/62825704" Ref="R?"  Part="1"
-AR Path="/62804339/62825704" Ref="R?"  Part="1"
-F 0 "R?" H 4570 4796 50  0000 L CNN
+AR Path="/62804339/62825704" Ref="R42"  Part="1"
+F 0 "R42" H 4570 4796 50  0000 L CNN
 F 1 "270" H 4570 4705 50  0000 L CNN
 F 2 "" V 4430 4750 50  0001 C CNN
@@
 P 3500 4250
 AR Path="/62740CD0/6282665D" Ref="R?"  Part="1"
-AR Path="/62804339/6282665D" Ref="R?"  Part="1"
-F 0 "R?" H 3570 4296 50  0000 L CNN
+AR Path="/62804339/6282665D" Ref="R44"  Part="1"
+F 0 "R44" H 3570 4296 50  0000 L CNN
 F 1 "22k" H 3570 4205 50  0000 L CNN
 F 2 "" V 3430 4250 50  0001 C CNN
@@
 P 3000 4250
 AR Path="/62740CD0/628267EC" Ref="R?"  Part="1"
-AR Path="/62804339/628267EC" Ref="R?"  Part="1"
-F 0 "R?" H 3070 4296 50  0000 L CNN
+AR Path="/62804339/628267EC" Ref="R45"  Part="1"
+F 0 "R45" H 3070 4296 50  0000 L CNN
 F 1 "22k" H 3070 4205 50  0000 L CNN
 F 2 "" V 2930 4250 50  0001 C CNN
@@
 P 2000 4250
 AR Path="/62740CD0/62826CDD" Ref="R?"  Part="1"
-AR Path="/62804339/62826CDD" Ref="R?"  Part="1"
-F 0 "R?" H 2070 4296 50  0000 L CNN
+AR Path="/62804339/62826CDD" Ref="R47"  Part="1"
+F 0 "R47" H 2070 4296 50  0000 L CNN
 F 1 "100k" H 2070 4205 50  0000 L CNN
 F 2 "" V 1930 4250 50  0001 C CNN
@@
 P 1500 4250
 AR Path="/62740CD0/62826FC4" Ref="R?"  Part="1"
-AR Path="/62804339/62826FC4" Ref="R?"  Part="1"
-F 0 "R?" H 1570 4296 50  0000 L CNN
+AR Path="/62804339/62826FC4" Ref="R48"  Part="1"
+F 0 "R48" H 1570 4296 50  0000 L CNN
 F 1 "33k" H 1570 4205 50  0000 L CNN
 F 2 "" V 1430 4250 50  0001 C CNN
@@
 P 2250 4000
 AR Path="/62740CD0/62829D12" Ref="R?"  Part="1"
-AR Path="/62804339/62829D12" Ref="R?"  Part="1"
-F 0 "R?" H 2320 4046 50  0000 L CNN
+AR Path="/62804339/62829D12" Ref="R46"  Part="1"
+F 0 "R46" H 2320 4046 50  0000 L CNN
 F 1 "33k" H 2320 3955 50  0000 L CNN
 F 2 "" V 2180 4000 50  0001 C CNN
@@
 P 2750 4000
 AR Path="/62740CD0/6282A3BB" Ref="D?"  Part="1"
-AR Path="/62804339/6282A3BB" Ref="D?"  Part="1"
-F 0 "D?" V 2796 3920 50  0000 R CNN
+AR Path="/62804339/6282A3BB" Ref="D4"  Part="1"
+F 0 "D4" V 2796 3920 50  0000 R CNN
 F 1 "D" V 2705 3920 50  0000 R CNN
 F 2 "" H 2750 4000 50  0001 C CNN
@@
 AR Path="/6276643A/6282AE47" Ref="Q?"  Part="1"
 AR Path="/62740CD0/6282AE47" Ref="Q?"  Part="1"
-AR Path="/62804339/6282AE47" Ref="Q?"  Part="1"
-F 0 "Q?" H 4591 4046 50  0000 L CNN
+AR Path="/62804339/6282AE47" Ref="Q6"  Part="1"
+F 0 "Q6" H 4591 4046 50  0000 L CNN
 F 1 "Q_NPN_BCE" H 4591 3955 50  0000 L CNN
 F 2 "" H 4600 4100 50  0001 C CNN

Commit message: Footprints added
Added most of the footprints for a 0805 SMD PCB. some placeholder footprints added and some missing
Parts:
- C25, C29, C30, C31, C32, C33: renamed from C?; footprint (none) -> Capacitor_SMD:C_0805_2012Metric_Pad1.18x1.45mm_HandSolder
- D4: footprint (none) -> Diode_SMD:D_SOD-123
- Q6: footprint (none) -> Package_TO_SOT_SMD:SOT-23
- R40, R41, R42, R43, R44, R45, R46, R47, R48: footprint (none) -> Resistor_SMD:R_0805_2012Metric_Pad1.20x1.40mm_HandSolder
Changed lines of the file:
@@
 F 0 "R41" H 4820 3546 50  0000 L CNN
 F 1 "47k" H 4820 3455 50  0000 L CNN
-F 2 "" V 4680 3500 50  0001 C CNN
+F 2 "Resistor_SMD:R_0805_2012Metric_Pad1.20x1.40mm_HandSolder" V 4680 3500 50  0001 C CNN
 F 3 "~" H 4750 3500 50  0001 C CNN
 	1    4750 3500
@@
 AR Path="/6276643A/6280F2C0" Ref="#PWR?"  Part="1"
 AR Path="/62740CD0/6280F2C0" Ref="#PWR?"  Part="1"
-AR Path="/62804339/6280F2C0" Ref="#PWR?"  Part="1"
-F 0 "#PWR?" H 1500 4250 50  0001 C CNN
+AR Path="/62804339/6280F2C0" Ref="#PWR0110"  Part="1"
+F 0 "#PWR0110" H 1500 4250 50  0001 C CNN
 F 1 "GND" H 1505 4327 50  0000 C CNN
 F 2 "" H 1500 4500 50  0001 C CNN
@@
 AR Path="/6276643A/6280F2D2" Ref="#PWR?"  Part="1"
 AR Path="/62740CD0/6280F2D2" Ref="#PWR?"  Part="1"
-AR Path="/62804339/6280F2D2" Ref="#PWR?"  Part="1"
-F 0 "#PWR?" H 4500 2850 50  0001 C CNN
+AR Path="/62804339/6280F2D2" Ref="#PWR0111"  Part="1"
+F 0 "#PWR0111" H 4500 2850 50  0001 C CNN
 F 1 "+6V" H 4515 3173 50  0000 C CNN
 F 2 "" H 4500 3000 50  0001 C CNN
@@
 F 0 "R40" H 4570 3296 50  0000 L CNN
 F 1 "10k" H 4570 3205 50  0000 L CNN
-F 2 "" V 4430 3250 50  0001 C CNN
+F 2 "Resistor_SMD:R_0805_2012Metric_Pad1.20x1.40mm_HandSolder" V 4430 3250 50  0001 C CNN
 F 3 "~" H 4500 3250 50  0001 C CNN
 	1    4500 3250
@@
 F 0 "R43" H 4070 3796 50  0000 L CNN
 F 1 "2.2M" H 4070 3705 50  0000 L CNN
-F 2 "" V 3930 3750 50  0001 C CNN
+F 2 "Resistor_SMD:R_0805_2012Metric_Pad1.20x1.40mm_HandSolder" V 3930 3750 50  0001 C CNN
 F 3 "~" H 4000 3750 50  0001 C CNN
 	1    4000 3750
@@
 F 0 "R42" H 4570 4796 50  0000 L CNN
 F 1 "270" H 4570 4705 50  0000 L CNN
-F 2 "" V 4430 4750 50  0001 C CNN
+F 2 "Resistor_SMD:R_0805_2012Metric_Pad1.20x1.40mm_HandSolder" V 4430 4750 50  0001 C CNN
 F 3 "~" H 4500 4750 50  0001 C CNN
 	1    4500 4750
@@
 F 0 "R44" H 3570 4296 50  0000 L CNN
 F 1 "22k" H 3570 4205 50  0000 L CNN
-F 2 "" V 3430 4250 50  0001 C CNN
+F 2 "Resistor_SMD:R_0805_2012Metric_Pad1.20x1.40mm_HandSolder" V 3430 4250 50  0001 C CNN
 F 3 "~" H 3500 4250 50  0001 C CNN
 	1    3500 4250
@@
 F 0 "R45" H 3070 4296 50  0000 L CNN
 F 1 "22k" H 3070 4205 50  0000 L CNN
-F 2 "" V 2930 4250 50  0001 C CNN
+F 2 "Resistor_SMD:R_0805_2012Metric_Pad1.20x1.40mm_HandSolder" V 2930 4250 50  0001 C CNN
 F 3 "~" H 3000 4250 50  0001 C CNN
 	1    3000 4250
@@
 F 0 "R47" H 2070 4296 50  0000 L CNN
 F 1 "100k" H 2070 4205 50  0000 L CNN
-F 2 "" V 1930 4250 50  0001 C CNN
+F 2 "Resistor_SMD:R_0805_2012Metric_Pad1.20x1.40mm_HandSolder" V 1930 4250 50  0001 C CNN
 F 3 "~" H 2000 4250 50  0001 C CNN
 	1    2000 4250
@@
 F 0 "R48" H 1570 4296 50  0000 L CNN
 F 1 "33k" H 1570 4205 50  0000 L CNN
-F 2 "" V 1430 4250 50  0001 C CNN
+F 2 "Resistor_SMD:R_0805_2012Metric_Pad1.20x1.40mm_HandSolder" V 1430 4250 50  0001 C CNN
 F 3 "~" H 1500 4250 50  0001 C CNN
 	1    1500 4250
@@
 AR Path="/6276643A/628275F6" Ref="C?"  Part="1"
 AR Path="/62740CD0/628275F6" Ref="C?"  Part="1"
-AR Path="/62804339/628275F6" Ref="C?"  Part="1"
-F 0 "C?" H 5365 3546 50  0000 L CNN
+AR Path="/62804339/628275F6" Ref="C25"  Part="1"
+F 0 "C25" H 5365 3546 50  0000 L CNN
 F 1 ".0022" H 5365 3455 50  0000 L CNN
-F 2 "" H 5288 3350 50  0001 C CNN
+F 2 "Capacitor_SMD:C_0805_2012Metric_Pad1.18x1.45mm_HandSolder" H 5288 3350 50  0001 C CNN
 F 3 "~" H 5250 3500 50  0001 C CNN
 	1    5250 3500
@@
 AR Path="/6276643A/62827C65" Ref="C?"  Part="1"
 AR Path="/62740CD0/62827C65" Ref="C?"  Part="1"
-AR Path="/62804339/62827C65" Ref="C?"  Part="1"
-F 0 "C?" H 3615 3546 50  0000 L CNN
+AR Path="/62804339/62827C65" Ref="C29"  Part="1"
+F 0 "C29" H 3615 3546 50  0000 L CNN
 F 1 ".0022" H 3615 3455 50  0000 L CNN
-F 2 "" H 3538 3350 50  0001 C CNN
+F 2 "Capacitor_SMD:C_0805_2012Metric_Pad1.18x1.45mm_HandSolder" H 3538 3350 50  0001 C CNN
 F 3 "~" H 3500 3500 50  0001 C CNN
 	1    3500 3500
@@
 AR Path="/6276643A/628283B5" Ref="C?"  Part="1"
 AR Path="/62740CD0/628283B5" Ref="C?"  Part="1"
-AR Path="/62804339/628283B5" Ref="C?"  Part="1"
-F 0 "C?" H 3365 4046 50  0000 L CNN
+AR Path="/62804339/628283B5" Ref="C30"  Part="1"
+F 0 "C30" H 3365 4046 50  0000 L CNN
 F 1 ".0015" H 3365 3955 50  0000 L CNN
-F 2 "" H 3288 3850 50  0001 C CNN
+F 2 "Capacitor_SMD:C_0805_2012Metric_Pad1.18x1.45mm_HandSolder" H 3288 3850 50  0001 C CNN
 F 3 "~" H 3250 4000 50  0001 C CNN
 	1    3250 4000
@@
 AR Path="/6276643A/62828526" Ref="C?"  Part="1"
 AR Path="/62740CD0/62828526" Ref="C?"  Part="1"
-AR Path="/62804339/62828526" Ref="C?"  Part="1"
-F 0 "C?" H 3865 4046 50  0000 L CNN
+AR Path="/62804339/62828526" Ref="C31"  Part="1"
+F 0 "C31" H 3865 4046 50  0000 L CNN
 F 1 ".0015" H 3865 3955 50  0000 L CNN
-F 2 "" H 3788 3850 50  0001 C CNN
+F 2 "Capacitor_SMD:C_0805_2012Metric_Pad1.18x1.45mm_HandSolder" H 3788 3850 50  0001 C CNN
 F 3 "~" H 3750 4000 50  0001 C CNN
 	1    3750 4000
@@
 AR Path="/6276643A/62828F17" Ref="C?"  Part="1"
 AR Path="/62740CD0/62828F17" Ref="C?"  Part="1"
-AR Path="/62804339/62828F17" Ref="C?"  Part="1"
-F 0 "C?" H 2615 4296 50  0000 L CNN
+AR Path="/62804339/62828F17" Ref="C32"  Part="1"
+F 0 "C32" H 2615 4296 50  0000 L CNN
 F 1 "47p" H 2615 4205 50  0000 L CNN
-F 2 "" H 2538 4100 50  0001 C CNN
+F 2 "Capacitor_SMD:C_0805_2012Metric_Pad1.18x1.45mm_HandSolder" H 2538 4100 50  0001 C CNN
 F 3 "~" H 2500 4250 50  0001 C CNN
 	1    2500 4250
@@
 AR Path="/6276643A/62829280" Ref="C?"  Part="1"
 AR Path="/62740CD0/62829280" Ref="C?"  Part="1"
-AR Path="/62804339/62829280" Ref="C?"  Part="1"
-F 0 "C?" H 1865 4046 50  0000 L CNN
+AR Path="/62804339/62829280" Ref="C33"  Part="1"
+F 0 "C33" H 1865 4046 50  0000 L CNN
 F 1 ".0027" H 1865 3955 50  0000 L CNN
-F 2 "" H 1788 3850 50  0001 C CNN
+F 2 "Capacitor_SMD:C_0805_2012Metric_Pad1.18x1.45mm_HandSolder" H 1788 3850 50  0001 C CNN
 F 3 "~" H 1750 4000 50  0001 C CNN
 	1    1750 4000
@@
 F 0 "R46" H 2320 4046 50  0000 L CNN
 F 1 "33k" H 2320 3955 50  0000 L CNN
-F 2 "" V 2180 4000 50  0001 C CNN
+F 2 "Resistor_SMD:R_0805_2012Metric_Pad1.20x1.40mm_HandSolder" V 2180 4000 50  0001 C CNN
 F 3 "~" H 2250 4000 50  0001 C CNN
 	1    2250 4000
@@
 F 0 "D4" V 2796 3920 50  0000 R CNN
 F 1 "D" V 2705 3920 50  0000 R CNN
-F 2 "" H 2750 4000 50  0001 C CNN
+F 2 "Diode_SMD:D_SOD-123" H 2750 4000 50  0001 C CNN
 F 3 "~" H 2750 4000 50  0001 C CNN
 	1    2750 4000
@@
 F 0 "Q6" H 4591 4046 50  0000 L CNN
 F 1 "Q_NPN_BCE" H 4591 3955 50  0000 L CNN
-F 2 "" H 4600 4100 50  0001 C CNN
+F 2 "Package_TO_SOT_SMD:SOT-23" H 4600 4100 50  0001 C CNN
 F 3 "~" H 4400 4000 50  0001 C CNN
 	1    4400 4000
@@
 AR Path="/6276643A/628334C8" Ref="#PWR?"  Part="1"
 AR Path="/62740CD0/628334C8" Ref="#PWR?"  Part="1"
-AR Path="/62804339/628334C8" Ref="#PWR?"  Part="1"
-F 0 "#PWR?" H 2000 4250 50  0001 C CNN
+AR Path="/62804339/628334C8" Ref="#PWR0112"  Part="1"
+F 0 "#PWR0112" H 2000 4250 50  0001 C CNN
 F 1 "GND" H 2005 4327 50  0000 C CNN
 F 2 "" H 2000 4500 50  0001 C CNN
@@
 AR Path="/6276643A/62833DAE" Ref="#PWR?"  Part="1"
 AR Path="/62740CD0/62833DAE" Ref="#PWR?"  Part="1"
-AR Path="/62804339/62833DAE" Ref="#PWR?"  Part="1"
-F 0 "#PWR?" H 2500 4250 50  0001 C CNN
+AR Path="/62804339/62833DAE" Ref="#PWR0113"  Part="1"
+F 0 "#PWR0113" H 2500 4250 50  0001 C CNN
 F 1 "GND" H 2505 4327 50  0000 C CNN
 F 2 "" H 2500 4500 50  0001 C CNN
@@
 AR Path="/6276643A/62833DB4" Ref="#PWR?"  Part="1"
 AR Path="/62740CD0/62833DB4" Ref="#PWR?"  Part="1"
-AR Path="/62804339/62833DB4" Ref="#PWR?"  Part="1"
-F 0 "#PWR?" H 3000 4250 50  0001 C CNN
+AR Path="/62804339/62833DB4" Ref="#PWR0114"  Part="1"
+F 0 "#PWR0114" H 3000 4250 50  0001 C CNN
 F 1 "GND" H 3005 4327 50  0000 C CNN
 F 2 "" H 3000 4500 50  0001 C CNN
@@
 AR Path="/6276643A/628348FE" Ref="#PWR?"  Part="1"
 AR Path="/62740CD0/628348FE" Ref="#PWR?"  Part="1"
-AR Path="/62804339/628348FE" Ref="#PWR?"  Part="1"
-F 0 "#PWR?" H 3500 4250 50  0001 C CNN
+AR Path="/62804339/628348FE" Ref="#PWR0115"  Part="1"
+F 0 "#PWR0115" H 3500 4250 50  0001 C CNN
 F 1 "GND" H 3505 4327 50  0000 C CNN
 F 2 "" H 3500 4500 50  0001 C CNN
@@
 AR Path="/6276643A/62834C57" Ref="#PWR?"  Part="1"
 AR Path="/62740CD0/62834C57" Ref="#PWR?"  Part="1"
-AR Path="/62804339/62834C57" Ref="#PWR?"  Part="1"
-F 0 "#PWR?" H 4500 4750 50  0001 C CNN
+AR Path="/62804339/62834C57" Ref="#PWR0116"  Part="1"
+F 0 "#PWR0116" H 4500 4750 50  0001 C CNN
 F 1 "GND" H 4505 4827 50  0000 C CNN
 F 2 "" H 4500 5000 50  0001 C CNN

Commit message: changed some stuff
Parts:
- C25, C29, C30, C31, C32, C33: footprint Capacitor_SMD:C_0805_2012Metric_Pad1.18x1.45mm_HandSolder -> Capacitor_SMD:C_0805_2012Metric
- D4: footprint Diode_SMD:D_SOD-123 -> Diode_SMD:D_SOD-123F
- Q6: footprint Package_TO_SOT_SMD:SOT-23 -> Package_TO_SOT_SMD:SOT-89-3
- R40, R41, R42, R43, R44, R45, R46, R47, R48: footprint Resistor_SMD:R_0805_2012Metric_Pad1.20x1.40mm_HandSolder -> Resistor_SMD:R_0805_2012Metric
Changed lines of the file:
@@
 $Descr A4 11693 8268
 encoding utf-8
-Sheet 3 7
+Sheet 3 8
 Title ""
 Date ""
@@
 F 0 "R41" H 4820 3546 50  0000 L CNN
 F 1 "47k" H 4820 3455 50  0000 L CNN
-F 2 "Resistor_SMD:R_0805_2012Metric_Pad1.20x1.40mm_HandSolder" V 4680 3500 50  0001 C CNN
+F 2 "Resistor_SMD:R_0805_2012Metric" V 4680 3500 50  0001 C CNN
 F 3 "~" H 4750 3500 50  0001 C CNN
 	1    4750 3500
@@
 F 0 "R40" H 4570 3296 50  0000 L CNN
 F 1 "10k" H 4570 3205 50  0000 L CNN
-F 2 "Resistor_SMD:R_0805_2012Metric_Pad1.20x1.40mm_HandSolder" V 4430 3250 50  0001 C CNN
+F 2 "Resistor_SMD:R_0805_2012Metric" V 4430 3250 50  0001 C CNN
 F 3 "~" H 4500 3250 50  0001 C CNN
 	1    4500 3250
@@
 F 0 "R43" H 4070 3796 50  0000 L CNN
 F 1 "2.2M" H 4070 3705 50  0000 L CNN
-F 2 "Resistor_SMD:R_0805_2012Metric_Pad1.20x1.40mm_HandSolder" V 3930 3750 50  0001 C CNN
+F 2 "Resistor_SMD:R_0805_2012Metric" V 3930 3750 50  0001 C CNN
 F 3 "~" H 4000 3750 50  0001 C CNN
 	1    4000 3750
@@
 F 0 "R42" H 4570 4796 50  0000 L CNN
 F 1 "270" H 4570 4705 50  0000 L CNN
-F 2 "Resistor_SMD:R_0805_2012Metric_Pad1.20x1.40mm_HandSolder" V 4430 4750 50  0001 C CNN
+F 2 "Resistor_SMD:R_0805_2012Metric" V 4430 4750 50  0001 C CNN
 F 3 "~" H 4500 4750 50  0001 C CNN
 	1    4500 4750
@@
 F 0 "R44" H 3570 4296 50  0000 L CNN
 F 1 "22k" H 3570 4205 50  0000 L CNN
-F 2 "Resistor_SMD:R_0805_2012Metric_Pad1.20x1.40mm_HandSolder" V 3430 4250 50  0001 C CNN
+F 2 "Resistor_SMD:R_0805_2012Metric" V 3430 4250 50  0001 C CNN
 F 3 "~" H 3500 4250 50  0001 C CNN
 	1    3500 4250
@@
 F 0 "R45" H 3070 4296 50  0000 L CNN
 F 1 "22k" H 3070 4205 50  0000 L CNN
-F 2 "Resistor_SMD:R_0805_2012Metric_Pad1.20x1.40mm_HandSolder" V 2930 4250 50  0001 C CNN
+F 2 "Resistor_SMD:R_0805_2012Metric" V 2930 4250 50  0001 C CNN
 F 3 "~" H 3000 4250 50  0001 C CNN
 	1    3000 4250
@@
 F 0 "R47" H 2070 4296 50  0000 L CNN
 F 1 "100k" H 2070 4205 50  0000 L CNN
-F 2 "Resistor_SMD:R_0805_2012Metric_Pad1.20x1.40mm_HandSolder" V 1930 4250 50  0001 C CNN
+F 2 "Resistor_SMD:R_0805_2012Metric" V 1930 4250 50  0001 C CNN
 F 3 "~" H 2000 4250 50  0001 C CNN
 	1    2000 4250
@@
 F 0 "R48" H 1570 4296 50  0000 L CNN
 F 1 "33k" H 1570 4205 50  0000 L CNN
-F 2 "Resistor_SMD:R_0805_2012Metric_Pad1.20x1.40mm_HandSolder" V 1430 4250 50  0001 C CNN
+F 2 "Resistor_SMD:R_0805_2012Metric" V 1430 4250 50  0001 C CNN
 F 3 "~" H 1500 4250 50  0001 C CNN
 	1    1500 4250
@@
 F 0 "C25" H 5365 3546 50  0000 L CNN
 F 1 ".0022" H 5365 3455 50  0000 L CNN
-F 2 "Capacitor_SMD:C_0805_2012Metric_Pad1.18x1.45mm_HandSolder" H 5288 3350 50  0001 C CNN
+F 2 "Capacitor_SMD:C_0805_2012Metric" H 5288 3350 50  0001 C CNN
 F 3 "~" H 5250 3500 50  0001 C CNN
 	1    5250 3500
@@
 F 0 "C29" H 3615 3546 50  0000 L CNN
 F 1 ".0022" H 3615 3455 50  0000 L CNN
-F 2 "Capacitor_SMD:C_0805_2012Metric_Pad1.18x1.45mm_HandSolder" H 3538 3350 50  0001 C CNN
+F 2 "Capacitor_SMD:C_0805_2012Metric" H 3538 3350 50  0001 C CNN
 F 3 "~" H 3500 3500 50  0001 C CNN
 	1    3500 3500
@@
 F 0 "C30" H 3365 4046 50  0000 L CNN
 F 1 ".0015" H 3365 3955 50  0000 L CNN
-F 2 "Capacitor_SMD:C_0805_2012Metric_Pad1.18x1.45mm_HandSolder" H 3288 3850 50  0001 C CNN
+F 2 "Capacitor_SMD:C_0805_2012Metric" H 3288 3850 50  0001 C CNN
 F 3 "~" H 3250 4000 50  0001 C CNN
 	1    3250 4000
@@
 F 0 "C31" H 3865 4046 50  0000 L CNN
 F 1 ".0015" H 3865 3955 50  0000 L CNN
-F 2 "Capacitor_SMD:C_0805_2012Metric_Pad1.18x1.45mm_HandSolder" H 3788 3850 50  0001 C CNN
+F 2 "Capacitor_SMD:C_0805_2012Metric" H 3788 3850 50  0001 C CNN
 F 3 "~" H 3750 4000 50  0001 C CNN
 	1    3750 4000
@@
 F 0 "C32" H 2615 4296 50  0000 L CNN
 F 1 "47p" H 2615 4205 50  0000 L CNN
-F 2 "Capacitor_SMD:C_0805_2012Metric_Pad1.18x1.45mm_HandSolder" H 2538 4100 50  0001 C CNN
+F 2 "Capacitor_SMD:C_0805_2012Metric" H 2538 4100 50  0001 C CNN
 F 3 "~" H 2500 4250 50  0001 C CNN
 	1    2500 4250
@@
 F 0 "C33" H 1865 4046 50  0000 L CNN
 F 1 ".0027" H 1865 3955 50  0000 L CNN
-F 2 "Capacitor_SMD:C_0805_2012Metric_Pad1.18x1.45mm_HandSolder" H 1788 3850 50  0001 C CNN
+F 2 "Capacitor_SMD:C_0805_2012Metric" H 1788 3850 50  0001 C CNN
 F 3 "~" H 1750 4000 50  0001 C CNN
 	1    1750 4000
@@
 F 0 "R46" H 2320 4046 50  0000 L CNN
 F 1 "33k" H 2320 3955 50  0000 L CNN
-F 2 "Resistor_SMD:R_0805_2012Metric_Pad1.20x1.40mm_HandSolder" V 2180 4000 50  0001 C CNN
+F 2 "Resistor_SMD:R_0805_2012Metric" V 2180 4000 50  0001 C CNN
 F 3 "~" H 2250 4000 50  0001 C CNN
 	1    2250 4000
@@
 F 0 "D4" V 2796 3920 50  0000 R CNN
 F 1 "D" V 2705 3920 50  0000 R CNN
-F 2 "Diode_SMD:D_SOD-123" H 2750 4000 50  0001 C CNN
+F 2 "Diode_SMD:D_SOD-123F" H 2750 4000 50  0001 C CNN
 F 3 "~" H 2750 4000 50  0001 C CNN
 	1    2750 4000
@@
 F 0 "Q6" H 4591 4046 50  0000 L CNN
 F 1 "Q_NPN_BCE" H 4591 3955 50  0000 L CNN
-F 2 "Package_TO_SOT_SMD:SOT-23" H 4600 4100 50  0001 C CNN
+F 2 "Package_TO_SOT_SMD:SOT-89-3" H 4600 4100 50  0001 C CNN
 F 3 "~" H 4400 4000 50  0001 C CNN
 	1    4400 4000
